File: pcb_v2/sr8a/sr8a.kicad_pcb (KiCad board)
At the start: 2 copper layers, 33.6 x 40.6 mm, 9 parts, among them J1 local_bus, U2 74LS374

Commit message: arquivos no note
Parts:
- moved D2 13.0 mm to (129.5, 76.2), turned to -90 degrees
- moved D1 12.9 mm to (129.5, 85.6), turned to 90 degrees
- moved R1 10.5 mm to (116.1, 85.9)
- moved R2 10.5 mm to (116.1, 80.0)
- moved C1 9.99 mm to (123.8, 64.1), turned to 90 degrees
- moved D3 8.89 mm to (129.5, 69.3)
- moved R3 8.76 mm to (123.7, 74.2)
- moved U2 0.18 mm to (119.9, 56.4)
Connections:
- D1 pad 1: GND -> Net-(D1-K)
- D1 pad 2: Net-(R1-Pad2) -> +5V
- D2 pad 1: Net-(D2-Pad1) -> GND
- D2 pad 2: +5V -> Net-(D2-A)
- J1 pad 13: n_read -> ~{read}
- J1 pad 27: n_read -> ~{read}
- R1 pad 1: write -> ~{read}
- R1 pad 2: Net-(R1-Pad2) -> Net-(D1-K)
- R2 pad 1: n_read -> write
- R2 pad 2: Net-(D2-Pad1) -> Net-(D2-A)
- U2 pad 1: n_read -> ~{read}
Routing:
- net ~{read}: track 0.00 -> 81.2 mm, vias 0 -> 2
- net n_read: track 72.4 -> 0.00 mm, vias 2 -> 0
- net +5V: track 60.0 -> 71.3 mm
- net GND: track 0.00 -> 10.2 mm
- net write: track 44.2 -> 53.0 mm
- net Net-(D2-A): track 0.00 -> 6.37 mm
- net Net-(R1-Pad2): track 6.24 -> 0.00 mm
- net Net-(D1-K): track 0.00 -> 5.95 mm
- net Net-(D2-Pad1): track 5.72 -> 0.00 mm
Other:
- board size 33.6 x 40.6 mm -> 43.5 x 40.6 mm
- board text added: "PWR"
- board text added: "RD"
- board text added: "WR"

Commit message: projeto enviado para impressao em dezembro/25
Parts:
- removed U2: 74LS374, Package_DIP:DIP-20_W7.62mm
- added U1: 74LS574, Package_DIP:DIP-20_W7.62mm, F.Cu at (99.7, 54.6)
- moved R1 23.4 mm to (111.8, 62.9)
- moved C1 15.3 mm to (111.8, 54.6), turned to -90 degrees
- moved R2 14.0 mm to (111.8, 66.7)
- moved D2 13.5 mm to (116.8, 80.7), turned to 90 degrees
- moved D3 13.4 mm to (116.8, 73.7), turned to 90 degrees
- moved D1 12.9 mm to (116.8, 87.6)
- moved R3 12.5 mm to (111.8, 70.5), turned to -90 degrees
Routing:
- net data_in_7: track 38.3 -> 13.4 mm, vias 1 -> 0
- net ~{read}: track 81.2 -> 58.8 mm, vias 2 -> 3
- net Net-(D1-K): track 5.95 -> 28.0 mm
- net data_in_6: track 34.5 -> 13.4 mm, vias 1 -> 0
- net data_in_0: track 30.2 -> 13.4 mm
- net data_in_1: track 28.1 -> 13.4 mm
- net data_in_5: track 25.6 -> 13.4 mm, vias 1 -> 0
- net data_out_7: track 33.0 -> 21.0 mm
- net write: track 53.0 -> 41.0 mm, vias 2 -> 1
- net data_out_0: track 32.5 -> 21.0 mm
- net data_in_2: track 22.2 -> 13.4 mm
- net data_in_3: track 21.2 -> 13.4 mm
- net Net-(D2-A): track 6.37 -> 14.1 mm
- net data_in_4: track 20.9 -> 13.4 mm, vias 1 -> 0
- net data_out_4: track 13.6 -> 21.0 mm
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Other:
- board size 43.5 x 40.6 mm -> 32.3 x 40.6 mm
- board text added: "Rev.A1 dezembro/2025"
- board text removed: "Rev.A1 julho/2025"
