File: pcb_v2/sr8a/sr8a.kicad_sch (KiCad schematic)
At the start: 9 parts, among them J1 local_bus, U1 74LS574

Commit message: arquivos no note
Parts:
- removed U1: 74LS574, Package_DIP:SMDIP-20_W7.62mm, symbol 74xx:74LS574
- added U2: 74LS374, Package_DIP:DIP-20_W7.62mm, symbol 74xx:74LS374
- C1: footprint Capacitor_SMD:C_1206_3216Metric -> Capacitor_THT:C_Disc_D5.1mm_W3.2mm_P5.00mm
- R1: renamed from R2; footprint Resistor_SMD:R_1206_3216Metric -> Resistor_THT:R_Axial_DIN0207_L6.3mm_D2.5mm_P7.62mm_Horizontal
- R2: renamed from R1; footprint Resistor_SMD:R_1206_3216Metric -> Resistor_THT:R_Axial_DIN0207_L6.3mm_D2.5mm_P7.62mm_Horizontal
- R3: footprint Resistor_SMD:R_1206_3216Metric -> Resistor_THT:R_Axial_DIN0207_L6.3mm_D2.5mm_P7.62mm_Horizontal
Connections:
- net +5V: now also D1.2 (A), U2.20 (VCC); no longer D2.2 (A)
- net GND: now also D2.1 (K), U2.10 (GND); no longer D1.1 (K)
- net data_in_0: now also U2.3 (D0)
- net data_in_1: now also U2.4 (D1)
- net data_in_2: now also U2.7 (D2)
- net data_in_3: now also U2.8 (D3)
- net data_in_4: now also U2.13 (D4)
- net data_in_5: now also U2.14 (D5)
- net data_in_6: now also U2.17 (D6)
- net data_in_7: now also U2.18 (D7)
- net data_out_0: now also U2.2 (O0)
- net data_out_1: now also U2.5 (O1)
- net data_out_2: now also U2.6 (O2)
- net data_out_3: now also U2.9 (O3)
- net data_out_4: now also U2.12 (O4)
- net data_out_5: now also U2.15 (O5)
- net data_out_6: now also U2.16 (O6)
- net data_out_7: now also U2.19 (O7)
- net write: now also U2.11 (Cp)
- net at R1.2: now also D1.1 (K); no longer D2.1 (K)
- net at R2.2: now also D2.2 (A); no longer D1.2 (A)
- net n_read renamed ~{read}
- net ~{read}: now also U2.1 (OE)
- no-connect marks 0 -> 4

Commit message: projeto enviado para impressao em dezembro/25
Parts:
- removed U2: 74LS374, Package_DIP:DIP-20_W7.62mm, symbol 74xx:74LS374
- added U1: 74LS574, Package_DIP:DIP-20_W7.62mm, symbol 74xx:74LS574
Connections:
- net +5V: now also U1.20 (VCC)
- net GND: now also U1.10 (GND)
- net data_in_0: now also U1.2 (D0)
- net data_in_1: now also U1.3 (D1)
- net data_in_2: now also U1.4 (D2)
- net data_in_3: now also U1.5 (D3)
- net data_in_4: now also U1.6 (D4)
- net data_in_5: now also U1.7 (D5)
- net data_in_6: now also U1.8 (D6)
- net data_in_7: now also U1.9 (D7)
- net data_out_0: now also U1.19 (Q0)
- net data_out_1: now also U1.18 (Q1)
- net data_out_2: now also U1.17 (Q2)
- net data_out_3: now also U1.16 (Q3)
- net data_out_4: now also U1.15 (Q4)
- net data_out_5: now also U1.14 (Q5)
- net data_out_6: now also U1.13 (Q6)
- net data_out_7: now also U1.12 (Q7)
- net write: now also U1.11 (Cp)
- net ~{read}: now also U1.1 (OE)
Changed lines of the file:
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@@
+	)
+	(junction
+		(at 44.45 67.31)
+		(diameter 0)
+		(color 0 0 0 0)
 	)
 	(junction
 		(at 109.22 63.5)
-		(diameter 0)
-		(color 0 0 0 0)
-	)
-	(junction
-		(at 44.45 67.31)
 		(diameter 0)
 		(color 0 0 0 0)
@@
 	)
 	(symbol
-		(lib_id "74xx:74LS374")
-		(at 44.45 46.99 0)
-		(unit 1)
-		(exclude_from_sim no)
-		(in_bom yes)
-		(on_board yes)
-		(dnp no)
-		(fields_autoplaced yes)
-		(property "Reference" "U2"
-			(at 46.4694 26.67 0)
-			(effects
-				(font
-					(size 1.27 1.27)
-				)
-				(justify left)
-			)
-		)
-		(property "Value" "74LS374"
-			(at 46.4694 29.21 0)
-			(effects
-				(font
-					(size 1.27 1.27)
-				)
-				(justify left)
-			)
-		)
-		(property "Footprint" "Package_DIP:DIP-20_W7.62mm"
-			(at 44.45 46.99 0)
-			(effects
-				(font
-					(size 1.27 1.27)
-				)
-				(hide yes)
-			)
-		)
-		(property "Datasheet" "http://www.ti.com/lit/gpn/sn74LS374"
-			(at 44.45 46.99 0)
-			(effects
-				(font
-					(size 1.27 1.27)
-				)
-				(hide yes)
-			)
-		)
-		(property "Description" ""
-			(at 44.45 46.99 0)
-			(effects
-				(font
-					(size 1.27 1.27)
-				)
-			)
-		)
-		(pin "1"
-		)
-		(pin "10"
-		)
-		(pin "11"
-		)
-		(pin "12"
-		)
-		(pin "13"
-		)
-		(pin "14"
-		)
-		(pin "15"
-		)
-		(pin "16"
-		)
-		(pin "17"
-		)
-		(pin "18"
-		)
-		(pin "19"
-		)
-		(pin "2"
-		)
-		(pin "20"
-		)
-		(pin "3"
-		)
-		(pin "4"
-		)
-		(pin "5"
-		)
-		(pin "6"
-		)
-		(pin "7"
-		)
-		(pin "8"
-		)
-		(pin "9"
-		)
-		(instances
-			(project ""
-				(path "/8ea830d9-a456-4a42-bd6f-7aaef78f7a83"
-					(reference "U2")
-					(unit 1)
-				)
-			)
-		)
-	)
-	(symbol
 		(lib_id "Device:R")
 		(at 179.07 72.39 90)
@@
 					(unit 1)
 				)
+			)
+		)
+	)
+	(symbol
+		(lib_id "74xx:74LS574")
+		(at 44.45 46.99 0)
+		(unit 1)
+		(exclude_from_sim no)
+		(in_bom yes)
+		(on_board yes)
+		(dnp no)
+		(fields_autoplaced yes)
+		(property "Reference" "U1"
+			(at 46.5933 26.67 0)
+			(effects
+				(font
+					(size 1.27 1.27)
+				)
+				(justify left)
+			)
+		)
+		(property "Value" "74LS574"
+			(at 46.5933 29.21 0)
+			(effects
+				(font
+					(size 1.27 1.27)
+				)
+				(justify left)
+			)
+		)
+		(property "Footprint" "Package_DIP:DIP-20_W7.62mm"
+			(at 44.45 46.99 0)
+			(effects
+				(font
+					(size 1.27 1.27)
+				)
+				(hide yes)
+			)
+		)
+		(property "Datasheet" "http://www.ti.com/lit/gpn/sn74LS574"
+			(at 44.45 46.99 0)
+			(effects
+				(font
+					(size 1.27 1.27)
+				)
+				(hide yes)
+			)
+		)
+		(property "Description" "8-bit Register, 3-state outputs"
+			(at 44.45 46.99 0)
+			(effects
+				(font
+					(size 1.27 1.27)
+				)
+				(hide yes)
+			)
+		)
+		(pin "9"
+		)
+		(pin "3"
+		)
+		(pin "17"
+		)
+		(pin "4"
+		)
+		(pin "13"
+		)
+		(pin "5"
+		)
+		(pin "6"
+		)
+		(pin "16"
+		)
+		(pin "12"
+		)
+		(pin "11"
+		)
+		(pin "1"
+		)
+		(pin "20"
+		)
+		(pin "19"
+		)
+		(pin "7"
+		)
+		(pin "18"
+		)
+		(pin "10"
+		)
+		(pin "2"
+		)
+		(pin "15"
+		)
+		(pin "8"
+		)
+		(pin "14"
+		)
+		(instances
+			(project ""
+				(path "/8ea830d9-a456-4a42-bd6f-7aaef78f7a83"
+					(reference "U1")
+					(unit 1)
+				)
