File: pcb_v2/ex16a/ex16a.kicad_sch (KiCad schematic)
At the start: 18 parts, among them U1 74LS125, U10 74LS244, U11 74LS244, U2 74LS193, U3 74LS138, U4 74LS08, U5 74LS06, U6 74LS08, U7 74LS244, U8 74LS244, U9 74LS244

Commit message: alterando os pinos de alimentacao no conector
Parts:
- removed U5: 74LS06, symbol 74xx:74LS06
- added C1, C4, C5, C6: 100nF, symbol Device:C
- added D1: LED, LED_THT:LED_D5.0mm, symbol Device:LED
- added J1: addr_decoder, edge_connector:edge-connector-44, symbol Connector_Generic:Conn_02x22_Top_Bottom
- added R1, R10, R11, R12, R13, R14, R15, R16, R17, R18, R2, R3, R4, R5, R6, R7, R8, R9: 10K, symbol Device:R
- added R19: 1K, Resistor_THT:R_Axial_DIN0207_L6.3mm_D2.5mm_P7.62mm_Horizontal, symbol Device:R
- added U5: 74LS04, symbol 74xx:74LS04
- renumbered C1 to C2, C2 to C3
Connections:
- net +5V: now also U1.14 (VCC), U4.14 (VCC), U6.14 (VCC), C1.2, C4.2, C5.2, C6.2, J1.30 (Pin_30), J1.8 (Pin_8), R1.1, R10.1, R11.1, R12.1, R13.1, R14.1, R15.1, R16.1, R17.1, R18.1, R19.2, R2.1, R3.1, R4.1, R5.1, R6.1, R7.1, R8.1, R9.1, U5.14 (VCC)
- net GND: now also U1.7 (GND), U4.7 (GND), U6.7 (GND), C1.1, C4.1, C5.1, C6.1, D1.1 (K), J1.31 (Pin_31), J1.9 (Pin_9), U5.7 (GND)
- net inc_one: now also J1.37 (Pin_37), R7.2
- net inc_two: now also J1.44 (Pin_44), R13.2
- net inc_zero: now also J1.28 (Pin_28), R6.2
- net pc_inc: now also J1.20 (Pin_20)
- net pcia_swap: now also J1.22 (Pin_22)
- net pclr_swap: now also J1.21 (Pin_21)
- net ~{addr_one}: now also J1.36 (Pin_36), R8.2
- net ~{addr_pc}: now also J1.19 (Pin_19)
- net ~{addr_two}: now also J1.43 (Pin_43), R14.2
- net ~{addr_zero}: now also J1.27 (Pin_27), R5.2
- net ~{sel_read_lrh}: now also J1.18 (Pin_18)
- net ~{sel_read_lrl}: now also J1.17 (Pin_17)
- net ~{sel_read_one_h}: now also J1.35 (Pin_35), R9.2
- net ~{sel_read_one_l}: now also J1.34 (Pin_34), R10.2
- net ~{sel_read_pch}: now also J1.6 (Pin_6)
- net ~{sel_read_pcl}: now also J1.5 (Pin_5)
- net ~{sel_read_two_h}: now also J1.42 (Pin_42), R15.2
- net ~{sel_read_two_l}: now also J1.41 (Pin_41), R16.2
- net ~{sel_read_zero_h}: now also J1.26 (Pin_26), R4.2
- net ~{sel_read_zero_l}: now also J1.25 (Pin_25), R3.2
- net ~{sel_write_lrh}: now also J1.4 (Pin_4)
- net ~{sel_write_lrl}: now also J1.3 (Pin_3)
- net ~{sel_write_one_h}: now also J1.33 (Pin_33), R11.2
- net ~{sel_write_one_l}: now also J1.32 (Pin_32), R12.2
- net ~{sel_write_pch}: now also J1.2 (Pin_2)
- net ~{sel_write_pcl}: now also J1.1 (Pin_1)
- net ~{sel_write_two_h}: now also J1.40 (Pin_40), R17.2
- net ~{sel_write_two_l}: now also J1.39 (Pin_39), R18.2
- net ~{sel_write_zero_h}: now also J1.24 (Pin_24), R2.2
- net ~{sel_write_zero_l}: now also J1.23 (Pin_23), R1.2
- net ~{swap_6}: now also U5.4
- net at U1.13, U1.4, U2.3 (QA)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: now also U5.1
- net at U3.9 (O6): now also U5.3
- net at U1.1, U1.10: now also U5.2
- net lr_at_0 renamed lr_at_zero
- net lr_at_1 renamed lr_at_one
- net lr_at_2 renamed lr_at_two
- net pc_at_0 renamed pc_at_zero
- net pc_at_1 renamed pc_at_one
- net pc_at_2 renamed pc_at_two
- new net: D1.2 (A), R19.1
- no-connect marks 19 -> 43
Other:
- moved on the sheet: C7, C8, C9, U1E, U4D, U4E, U6D, U6E, U7, U8, U9

Commit message: concluido o desenho das placas satelite do banco de registradores de 16 bits
Parts:
- C1, C10, C11, C2, C3, C4, C5, C6, C7, C8, C9: footprint (none) -> Capacitor_THT:C_Disc_D5.1mm_W3.2mm_P5.00mm
- D1: value LED -> PWR
- R1, R10, R11, R12, R13, R14, R15, R16, R17, R18, R2, R3, R4, R5, R6, R7, R8, R9: footprint (none) -> Resistor_THT:R_Axial_DIN0207_L6.3mm_D2.5mm_P7.62mm_Horizontal
- U1, U4, U5, U6: footprint (none) -> Package_DIP:DIP-14_W7.62mm
- U10, U11, U7, U8, U9: footprint (none) -> Package_DIP:DIP-20_W7.62mm
- U2, U3: footprint (none) -> Package_DIP:DIP-16_W7.62mm
Connections:
- net +5V: now also J1.1 (Pin_1), J1.23 (Pin_23); no longer J1.30 (Pin_30), J1.8 (Pin_8)
- net GND: now also J1.22 (Pin_22), J1.44 (Pin_44); no longer J1.31 (Pin_31), J1.9 (Pin_9)
- net inc_two: now also J1.43 (Pin_43); no longer J1.44 (Pin_44)
- net inc_zero: now also J1.29 (Pin_29); no longer J1.28 (Pin_28)
- net pc_inc: now also J1.19 (Pin_19); no longer J1.20 (Pin_20)
- net pcia_swap: now also J1.21 (Pin_21); no longer J1.22 (Pin_22)
- net pclr_swap: now also J1.20 (Pin_20); no longer J1.21 (Pin_21)
- net ~{addr_pc}: now also J1.18 (Pin_18); no longer J1.19 (Pin_19)
- net ~{addr_two}: now also J1.42 (Pin_42); no longer J1.43 (Pin_43)
- net ~{addr_zero}: now also J1.28 (Pin_28); no longer J1.27 (Pin_27)
- net ~{sel_read_lrh}: now also J1.17 (Pin_17); no longer J1.18 (Pin_18)
- net ~{sel_read_lrl}: now also J1.16 (Pin_16); no longer J1.17 (Pin_17)
- net ~{sel_read_pch}: now also J1.7 (Pin_7); no longer J1.6 (Pin_6)
- net ~{sel_read_pcl}: now also J1.6 (Pin_6); no longer J1.5 (Pin_5)
- net ~{sel_read_two_h}: now also J1.41 (Pin_41); no longer J1.42 (Pin_42)
- net ~{sel_read_two_l}: now also J1.40 (Pin_40); no longer J1.41 (Pin_41)
- net ~{sel_read_zero_h}: now also J1.27 (Pin_27); no longer J1.26 (Pin_26)
- net ~{sel_read_zero_l}: now also J1.26 (Pin_26); no longer J1.25 (Pin_25)
- net ~{sel_write_lrh}: now also J1.5 (Pin_5); no longer J1.4 (Pin_4)
- net ~{sel_write_lrl}: now also J1.4 (Pin_4); no longer J1.3 (Pin_3)
- net ~{sel_write_pch}: now also J1.3 (Pin_3); no longer J1.2 (Pin_2)
- net ~{sel_write_pcl}: now also J1.2 (Pin_2); no longer J1.1 (Pin_1)
- net ~{sel_write_two_h}: now also J1.39 (Pin_39); no longer J1.40 (Pin_40)
- net ~{sel_write_two_l}: now also J1.38 (Pin_38); no longer J1.39 (Pin_39)
- net ~{sel_write_zero_h}: now also J1.25 (Pin_25); no longer J1.24 (Pin_24)
- net ~{sel_write_zero_l}: now also J1.24 (Pin_24); no longer J1.23 (Pin_23)
