File: pcb_v2/ula8-shiftera/ula8-shiftera.kicad_sch (KiCad schematic)
At the start: 17 parts, among them J1 ula8a, U1 74LS244, U2 74LS244, U3 74LS157, U4 74LS157

Commit message: revisao completa; mgrfa agora inclui sr8 e sgrda; remover estes dois no proximo commit
Parts:
- U3, U4: footprint (none) -> Package_DIP:DIP-16_W7.62mm
Connections:
- net +5V: now also J1.1 (Pin_1), J1.23 (Pin_23), U3.10 (I1c), U3.11 (I0c), U3.13 (I1d), U3.14 (I0d), U4.13 (I1d), U4.14 (I0d); no longer J1.10 (Pin_10), J1.32 (Pin_32)
- net GND: now also J1.22 (Pin_22), J1.44 (Pin_44), U3.5 (I0b); no longer J1.11 (Pin_11), J1.33 (Pin_33)
- net carry_in: now also J1.24 (Pin_24), U3.2 (I0a); no longer J1.23 (Pin_23), U3.11 (I0c), U3.14 (I0d)
- net lower_bus0: now also J1.2 (Pin_2), U3.6 (I1b); no longer J1.1 (Pin_1), U3.13 (I1d)
- net lower_bus1: now also J1.3 (Pin_3); no longer J1.2 (Pin_2)
- net lower_bus2: now also J1.4 (Pin_4); no longer J1.3 (Pin_3)
- net lower_bus3: now also J1.5 (Pin_5); no longer J1.4 (Pin_4)
- net lower_bus4: now also J1.6 (Pin_6); no longer J1.5 (Pin_5)
- net lower_bus5: now also J1.7 (Pin_7); no longer J1.6 (Pin_6)
- net lower_bus6: now also J1.8 (Pin_8); no longer J1.7 (Pin_7)
- net lower_bus7: now also J1.9 (Pin_9), U3.3 (I1a); no longer J1.8 (Pin_8), U3.10 (I1c)
- net option_rigth: now also J1.13 (Pin_13); no longer J1.16 (Pin_16)
- net option_rotate: now also J1.14 (Pin_14); no longer J1.17 (Pin_17)
- net ula_bus0: now also J1.36 (Pin_36); no longer J1.37 (Pin_37)
- net ula_bus1: now also J1.37 (Pin_37); no longer J1.38 (Pin_38)
- net ula_bus2: now also J1.38 (Pin_38); no longer J1.39 (Pin_39)
- net ula_bus3: now also J1.39 (Pin_39); no longer J1.40 (Pin_40)
- net ula_bus4: now also J1.40 (Pin_40); no longer J1.41 (Pin_41)
- net ula_bus5: now also J1.41 (Pin_41); no longer J1.42 (Pin_42)
- net ula_bus6: now also J1.42 (Pin_42); no longer J1.43 (Pin_43)
- net ula_bus7: now also J1.43 (Pin_43); no longer J1.44 (Pin_44)
- net n_select renamed ~{select}
- net ~{select}: now also J1.17 (Pin_17); no longer J1.15 (Pin_15)
- net n_shift_left renamed ~{shift_left}
- net n_shift_right renamed ~{shift_right}
- no-connect marks 28 -> 22

Commit message: deslocando alimentação para as estremidades do conector; carry out em três estados (ativo apenas quando select)
Parts:
- added C5, C6, C7: 100nF, Capacitor_THT:C_Disc_D5.1mm_W3.2mm_P5.00mm, symbol Device:C
- added U5: 74LS125, Package_DIP:DIP-14_W7.62mm, symbol 74xx:74LS125
- added U6, U7, U8: 74LS244, Package_DIP:DIP-20_W7.62mm, symbol 74xx:74LS244
Connections:
- net +5V: now also C5.2, C6.2, C7.2, U5.1, U5.10, U5.14 (VCC), U5.2, U5.4, U5.5, U5.9, U6.20 (VCC), U7.20 (VCC)
- net GND: now also C5.1, C6.1, C7.1, U5.7 (GND), U6.10 (GND), U7.10 (GND)
- net carry_out: now also U5.11; no longer U4.4 (Za)
- net lower_bus0: now also U6.4 (I1a)
- net lower_bus1: now also U6.6 (I2a), U7.2 (I0a)
- net lower_bus2: now also U6.8 (I3a), U7.4 (I1a)
- net lower_bus3: now also U6.11 (I0b), U7.6 (I2a)
- net lower_bus4: now also U6.13 (I1b), U7.8 (I3a)
- net lower_bus5: now also U6.15 (I2b), U7.11 (I0b)
- net lower_bus6: now also U6.17 (I3b), U7.13 (I1b)
- net lower_bus7: now also U7.15 (I2b)
- net ula_bus0: now also U6.18 (O0a), U7.18 (O0a)
- net ula_bus1: now also U6.16 (O1a), U7.16 (O1a)
- net ula_bus2: now also U6.14 (O2a), U7.14 (O2a)
- net ula_bus3: now also U6.12 (O3a), U7.12 (O3a)
- net ula_bus4: now also U6.9 (O0b), U7.9 (O0b)
- net ula_bus5: now also U6.7 (O1b), U7.7 (O1b)
- net ula_bus6: now also U6.5 (O2b), U7.5 (O2b)
- net ula_bus7: now also U6.3 (O3b), U7.3 (O3b)
- net ~{select}: now also U5.13
- net ~{shift_left}: now also U6.1 (OEa), U6.19 (OEb)
- net ~{shift_right}: now also U7.1 (OEa), U7.19 (OEb)
- net option_rigth renamed option_right
- new net: U4.4 (Za), U5.12
- new net new_bit_0: U6.2 (I0a), U7.17 (I3b)
- no-connect marks 22 -> 25
Other:
- moved on the sheet: C1, C2, C3, C4, U1, U2, U3, U4

Commit message: faltava salvar
Parts:
- removed C6, C7: 100nF, Capacitor_THT:C_Disc_D5.1mm_W3.2mm_P5.00mm, symbol Device:C
- removed U6, U7, U8: 74LS244, Package_DIP:DIP-20_W7.62mm, symbol 74xx:74LS244
Other:
- moved on the sheet: C1, C2, C3, C4, U1, U2, U3, U4, U5D
