File: pcb_v2/ula8-xora/ula8-xora.kicad_sch (KiCad schematic)
At the start: 11 parts, among them J1 ula8a, U3 74LS244

Commit message: revisao completa; mgrfa agora inclui sr8 e sgrda; remover estes dois no proximo commit
Parts:
- U1, U2: value (none) -> 74LS86; footprint (none) -> Package_DIP:DIP-14_W7.62mm
Connections:
- net +5V: now also J1.1 (Pin_1), J1.23 (Pin_23); no longer J1.10 (Pin_10), J1.32 (Pin_32)
- net GND: now also J1.22 (Pin_22), J1.44 (Pin_44); no longer J1.11 (Pin_11), J1.33 (Pin_33)
- net carry: now also J1.24 (Pin_24); no longer J1.23 (Pin_23)
- net lower_bus0: now also J1.2 (Pin_2); no longer J1.1 (Pin_1)
- net lower_bus1: now also J1.3 (Pin_3); no longer J1.2 (Pin_2)
- net lower_bus2: now also J1.4 (Pin_4); no longer J1.3 (Pin_3)
- net lower_bus3: now also J1.5 (Pin_5); no longer J1.4 (Pin_4)
- net lower_bus4: now also J1.6 (Pin_6); no longer J1.5 (Pin_5)
- net lower_bus5: now also J1.7 (Pin_7); no longer J1.6 (Pin_6)
- net lower_bus6: now also J1.8 (Pin_8); no longer J1.7 (Pin_7)
- net lower_bus7: now also J1.9 (Pin_9); no longer J1.8 (Pin_8)
- net ula_bus0: now also J1.36 (Pin_36); no longer J1.37 (Pin_37)
- net ula_bus1: now also J1.37 (Pin_37); no longer J1.38 (Pin_38)
- net ula_bus2: now also J1.38 (Pin_38); no longer J1.39 (Pin_39)
- net ula_bus3: now also J1.39 (Pin_39); no longer J1.40 (Pin_40)
- net ula_bus4: now also J1.40 (Pin_40); no longer J1.41 (Pin_41)
- net ula_bus5: now also J1.41 (Pin_41); no longer J1.42 (Pin_42)
- net ula_bus6: now also J1.42 (Pin_42); no longer J1.43 (Pin_43)
- net ula_bus7: now also J1.43 (Pin_43); no longer J1.44 (Pin_44)
- net upper_bus0: now also J1.25 (Pin_25); no longer J1.24 (Pin_24)
- net upper_bus1: now also J1.26 (Pin_26); no longer J1.25 (Pin_25)
- net upper_bus2: now also J1.27 (Pin_27); no longer J1.26 (Pin_26)
- net upper_bus3: now also J1.28 (Pin_28); no longer J1.27 (Pin_27)
- net upper_bus4: now also J1.29 (Pin_29); no longer J1.28 (Pin_28)
- net upper_bus5: now also J1.30 (Pin_30); no longer J1.29 (Pin_29)
- net upper_bus6: now also J1.31 (Pin_31); no longer J1.30 (Pin_30)
- net upper_bus7: now also J1.32 (Pin_32); no longer J1.31 (Pin_31)
- net ~{select}: now reaches J1.16 (Pin_16)
- net ~{select}: now also R2.2, U3.1 (OEa), U3.19 (OEb)
- removed net n_select: J1.15 (Pin_15), R2.2, U3.1 (OEa), U3.19 (OEb)

Commit message: carry out depende de select
Parts:
- added C4: 100nF, Capacitor_THT:C_Disc_D5.1mm_W3.2mm_P5.00mm, symbol Device:C
- added U4: 74LS125, Package_DIP:DIP-14_W7.62mm, symbol 74xx:74LS125
Connections:
- net +5V: now also C4.2, U4.10, U4.12, U4.13, U4.14 (VCC), U4.4, U4.5, U4.9
- net GND: now also C4.1, U4.7 (GND)
- net ~{select}: now also U4.1
- net carry renamed carry_in
- net carry_in: now also U4.2; no longer J1.35 (Pin_35)
- new net carry_out: J1.35 (Pin_35), U4.3
- no-connect marks 13 -> 16
Other:
- moved on the sheet: C1, C2, C3
