File: pcb_v2/ula8da/ula8da.kicad_sch (KiCad schematic)
At the start: 28 parts, among them J1 addr_decoder, J2 Conn_01x07, J3 Conn_01x07, J4 Conn_01x07, J5 Conn_01x07, Q1 BC548, U1 74LS138, U2 74HC238, U3 74HC238, U4 74HC238, U5 74LS04, U6 74LS244, U7 74LS04, U8 MC14495P, U9 SA39-11EWA

Commit message: PCB concluída
Parts:
- removed C7, C8: 100nF, Capacitor_THT:C_Disc_D5.1mm_W3.2mm_P5.00mm, symbol Device:C
- removed D2: LED, LED_THT:LED_D5.0mm, symbol Device:LED
- removed J2, J3, J4, J5: Conn_01x07, Connector_PinHeader_2.54mm:PinHeader_1x07_P2.54mm_Vertical, symbol Connector_Generic:Conn_01x07
- removed Q1: BC548, Package_TO_SOT_THT:TO-92_Inline, symbol Transistor_BJT:BC548
- removed U3, U4: 74HC238, Package_DIP:DIP-16_W7.62mm, symbol 74xx:74HC238
- removed U6: 74LS244, Package_DIP:DIP-20_W7.62mm, symbol 74xx:74LS244
- removed U7: 74LS04, Package_DIP:DIP-14_W7.62mm, symbol 74xx:74LS04
- removed U8: MC14495P, Package_DIP:DIP-16_W7.62mm, symbol Driver_LED:MC14495P
- removed U9: SA39-11EWA, Display_7Segment:Sx39-1xxxxx, symbol Display_Character:SA39-11EWA
- added D1, D10, D100, D101, D102, D103, D104, D105, D106, D107, D108, D109, D11, D110, D111, D112, D12, D13, D14, D15, D16, D17, D18, D19, D2, D20, D21, D22, D23, D24, D25, D26, D27, D28, D29, D3, D30, D31, D32, D33, D34, D35, D36, D37, D38, D39, D4, D40, D41, D42, D43, D44, D45, D46, D47, D48, D49, D5, D50, D51, D52, D53, D54, D55, D56, D57, D58, D59, D6, D60, D61, D62, D63, D64, D65, D66, D67, D68, D69, D7, D70, D71, D72, D73, D74, D75, D76, D77, D78, D79, D8, D80, D81, D82, D83, D84, D85, D86, D87, D88, D89, D9, D90, D91, D92, D93, D94, D95, D96, D97, D98, D99: 1N4148, Diode_THT:D_DO-35_SOD27_P3.81mm_Vertical_KathodeUp, symbol Diode:1N4148
- added D121, D122: LED, LED_THT:LED_D5.0mm, symbol Device:LED
- added R1, R4, R5, R6, R7, R8: 10K, Resistor_THT:R_Axial_DIN0207_L6.3mm_D2.5mm_P7.62mm_Horizontal, symbol Device:R
- added R121, R122: 1K, Resistor_THT:R_Axial_DIN0207_L6.3mm_D2.5mm_P7.62mm_Horizontal, symbol Device:R
- added U3, U4, U6: 74LS138, Package_DIP:DIP-16_W7.62mm, symbol 74xx:74LS138
- R2: value 1K -> 10K
- renumbered D1 to D120, R1 to R120
Connections:
- net clrif is gone; now on net ~{select_sx}: J1.28 (Pin_28)
- net right/set is gone; now on net rotate/value: J1.3 (Pin_3)
- net rotate/clear is gone; now on net invert_lower_bus: J1.2 (Pin_2)
- net setif is gone; now on net invert_upper_bus: J1.6 (Pin_6)
- net +5V: now also C6.2, J1.1 (Pin_1), J1.23 (Pin_23), R120.1, R2.2, R3.2, R1.2, R4.2, R5.2, R6.2, R7.2, R8.2, U3.16 (VCC), U4.16 (VCC), U6.16 (VCC); no longer C6.1, D120.2 (A), J1.14 (Pin_14), J1.36 (Pin_36)
- net GND: now also C6.1, D120.1 (K), J1.22 (Pin_22), J1.44 (Pin_44), D121.1 (K), D122.1 (K), U3.8 (GND), U4.8 (GND), U6.4 (E1), U6.5 (E2), U6.8 (GND); no longer C6.2, J1.15 (Pin_15), J1.37 (Pin_37), R120.2, R2.2
- net invert_lower_bus: now also U5.10; no longer J1.1 (Pin_1)
- net invert_ula_bus: now also J1.5 (Pin_5), U5.12; no longer J1.4 (Pin_4)
- net invert_upper_bus: now also U5.8; no longer J1.5 (Pin_5)
- net rd_addr_0: now also J1.19 (Pin_19); no longer J1.20 (Pin_20)
- net rd_addr_1: now also J1.20 (Pin_20); no longer J1.21 (Pin_21)
- net rd_addr_2: now also J1.40 (Pin_40); no longer J1.41 (Pin_41)
- net rd_addr_3: now also J1.41 (Pin_41); no longer J1.42 (Pin_42)
- net rd_addr_4: now also J1.42 (Pin_42), U1.4 (E1); no longer J1.43 (Pin_43)
- net ula_enable: now also J1.33 (Pin_33), R122.1, U3.6 (E3), U4.6 (E3), U6.6 (E3); no longer J1.32 (Pin_32), R3.2, U1.4 (E1)
- net wr_addr_0: now also J1.30 (Pin_30), U3.1 (A0), U4.1 (A0); no longer J1.29 (Pin_29)
- net wr_addr_1: now also J1.31 (Pin_31), U3.2 (A1), U4.2 (A1); no longer J1.30 (Pin_30)
- net wr_addr_2: now also J1.32 (Pin_32), U3.3 (A2), U4.3 (A2); no longer J1.31 (Pin_31)
- net wr_addr_3: now also U5.1, U3.4 (E1), U3.5 (E2); no longer U2.6 (E3), U5.9
- net ~{read_acc}: now also J1.21 (Pin_21); no longer J1.22 (Pin_22)
- net ~{read_psw}: now also J1.43 (Pin_43); no longer J1.44 (Pin_44)
- net ~{select_adder}: now also J1.26 (Pin_26), U6.15 (O0); no longer J1.25 (Pin_25)
- net ~{select_bitwise}: now also J1.24 (Pin_24), U6.14 (O1); no longer J1.23 (Pin_23)
- net ~{select_shifter}: now also J1.27 (Pin_27), U6.12 (O3); no longer J1.26 (Pin_26)
- net ~{select_sx}: now also U6.11 (O4); no longer J1.27 (Pin_27)
- net ~{select_xor}: now also J1.25 (Pin_25), U6.13 (O2); no longer J1.24 (Pin_24)
- net at U5.5: now also R2.1, D10.2 (A), D106.2 (A), D18.2 (A), D2.2 (A), D26.2 (A), D34.2 (A), D42.2 (A), D50.2 (A), D58.2 (A), D66.2 (A), D74.2 (A), D82.2 (A), D90.2 (A), D98.2 (A)
- net right/mode: now reaches U5.6
- net right/mode: now also J1.4 (Pin_4)
- net ~{wr_addr_3}: now reaches U5.2
- net ~{wr_addr_3}: now also U2.4 (~{E1}), U4.4 (E1), U4.5 (E2)
- net at U5.11: now also D100.2 (A), D108.2 (A), D12.2 (A), D20.2 (A), D28.2 (A), D36.2 (A), D4.2 (A), D44.2 (A), D52.2 (A), D60.2 (A), D68.2 (A), D76.2 (A), D84.2 (A), D92.2 (A), R4.1
- net at U5.3: now also D1.2 (A), D105.2 (A), D17.2 (A), D25.2 (A), D33.2 (A), D41.2 (A), D49.2 (A), D57.2 (A), D65.2 (A), D73.2 (A), D81.2 (A), D89.2 (A), D9.2 (A), D97.2 (A), R1.1
- net rotate/value: now reaches U5.4
- net at R3.1: now also U5.9, D107.2 (A), D11.2 (A), D19.2 (A), D27.2 (A), D3.2 (A), D35.2 (A), D43.2 (A), D51.2 (A), D59.2 (A), D67.2 (A), D75.2 (A), D83.2 (A), D91.2 (A), D99.2 (A)
- net at U5.13: now also D101.2 (A), D109.2 (A), D13.2 (A), D21.2 (A), D29.2 (A), D37.2 (A), D45.2 (A), D5.2 (A), D53.2 (A), D61.2 (A), D69.2 (A), D77.2 (A), D85.2 (A), D93.2 (A), R5.1
- net write_clock renamed write_enable
- net write_enable: now also U2.6 (E3), R121.1
- new net: D120.2 (A), R120.2
- new net: D103.2 (A), D111.2 (A), D15.2 (A), D23.2 (A), D31.2 (A), D39.2 (A), D47.2 (A), D55.2 (A), D63.2 (A), D7.2 (A), D71.2 (A), D79.2 (A), D87.2 (A), D95.2 (A), R7.1, U6.2 (A1)
- new net: D104.2 (A), D112.2 (A), D16.2 (A), D24.2 (A), D32.2 (A), D40.2 (A), D48.2 (A), D56.2 (A), D64.2 (A), D72.2 (A), D8.2 (A), D80.2 (A), D88.2 (A), D96.2 (A), R8.1, U6.1 (A0)
- new net: D102.2 (A), D110.2 (A), D14.2 (A), D22.2 (A), D30.2 (A), D38.2 (A), D46.2 (A), D54.2 (A), D6.2 (A), D62.2 (A), D70.2 (A), D78.2 (A), D86.2 (A), D94.2 (A), R6.1, U6.3 (A2)
- new net: D121.2 (A), R121.2
- new net: D122.2 (A), R122.2
- new net ~{do_add}: D1.1 (K), D2.1 (K), D3.1 (K), D4.1 (K), D5.1 (K), D6.1 (K), D7.1 (K), D8.1 (K), U3.15 (O0)
- new net ~{do_and}: D25.1 (K), D26.1 (K), D27.1 (K), D28.1 (K), D29.1 (K), D30.1 (K), D31.1 (K), D32.1 (K), U3.12 (O3)
- new net ~{do_clrcf}: D105.1 (K), D106.1 (K), D107.1 (K), D108.1 (K), D109.1 (K), D110.1 (K), D111.1 (K), D112.1 (K), U4.10 (O5)
- new net ~{do_cmp}: D17.1 (K), D18.1 (K), D19.1 (K), D20.1 (K), D21.1 (K), D22.1 (K), D23.1 (K), D24.1 (K), U3.13 (O2)
- new net ~{do_not}: D49.1 (K), D50.1 (K), D51.1 (K), D52.1 (K), D53.1 (K), D54.1 (K), D55.1 (K), D56.1 (K), U3.9 (O6)
- new net ~{do_or}: D33.1 (K), D34.1 (K), D35.1 (K), D36.1 (K), D37.1 (K), D38.1 (K), D39.1 (K), D40.1 (K), U3.11 (O4)
- new net ~{do_rol}: D81.1 (K), D82.1 (K), D83.1 (K), D84.1 (K), D85.1 (K), D86.1 (K), D87.1 (K), D88.1 (K), U4.13 (O2)
- new net ~{do_ror}: D73.1 (K), D74.1 (K), D75.1 (K), D76.1 (K), D77.1 (K), D78.1 (K), D79.1 (K), D80.1 (K), U4.14 (O1)
- new net ~{do_setcf}: D100.1 (K), D101.1 (K), D102.1 (K), D103.1 (K), D104.1 (K), D97.1 (K), D98.1 (K), D99.1 (K), U4.11 (O4)
- new net ~{do_shl}: D65.1 (K), D66.1 (K), D67.1 (K), D68.1 (K), D69.1 (K), D70.1 (K), D71.1 (K), D72.1 (K), U4.15 (O0)
- new net ~{do_shr}: D57.1 (K), D58.1 (K), D59.1 (K), D60.1 (K), D61.1 (K), D62.1 (K), D63.1 (K), D64.1 (K), U3.7 (O7)
- new net ~{do_sub}: D10.1 (K), D11.1 (K), D12.1 (K), D13.1 (K), D14.1 (K), D15.1 (K), D16.1 (K), D9.1 (K), U3.14 (O1)
- new net ~{do_sx}: D89.1 (K), D90.1 (K), D91.1 (K), D92.1 (K), D93.1 (K), D94.1 (K), D95.1 (K), D96.1 (K), U4.12 (O3)
- new net ~{do_xor}: D41.1 (K), D42.1 (K), D43.1 (K), D44.1 (K), D45.1 (K), D46.1 (K), D47.1 (K), D48.1 (K), U3.10 (O5)
- new net ~{select_cf}: J1.29 (Pin_29), U6.10 (O5)
- no-connect marks 43 -> 29
Other:
- moved on the sheet: C4, D120, R120, U5B, U5C
