File: pcb_v2/testbench-sub8/testbench-sub8.kicad_pcb (KiCad board)
At the start: 2 copper layers, 91.4 x 53.9 mm, 25 parts, among them J3 conn, U1 74LS574, U2 74LS574, U3 74LS240, U4 74LS125, U5 74LS125, U6 74LS125, U7 74LS125

Commit message: correção no valor do resitor do led de power
Parts:
- R9: value 10K -> 1K
Changed lines of the file:
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@@
 			)
 		)
-		(property "Value" "10K"
+		(property "Value" "1K"
 			(at 3.81 1.92 90)
 			(layer "F.Fab")
