File: pcb_v2/testbench/testbench.kicad_pcb (KiCad board)
At the start: 2 copper layers, 274.3 x 124.5 mm, 70 parts, among them J1 test_A, J10 test_C1, J11 test_C2, J12 test_C3, J15 lcd, J17 DEBUG, J18 power_jack, J2 test_B, J3 sub_0, J4 sub_8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

Commit message: ajuste no espacamento entre os conectores flat
Parts:
- moved J10 12.1 mm to (280.0, 46.4)
- moved J11 7.62 mm to (280.0, 76.2)
- moved J12 3.17 mm to (280.0, 106.0)
Routing:
- net test_power_vcc: track 236.2 -> 252.5 mm
- net test_25: track 114.7 -> 125.6 mm
- net test_1: track 102.8 -> 113.4 mm
- net test_2: track 103.1 -> 113.7 mm
- net test_26: track 115.8 -> 126.0 mm
- net test_3: track 103.5 -> 113.7 mm
- net test_4: track 99.2 -> 109.1 mm
- net test_27: track 116.9 -> 126.7 mm
- net test_6: track 100.8 -> 110.6 mm
- net test_5: track 99.6 -> 109.1 mm
- net test_28: track 113.1 -> 122.6 mm
- net test_29: track 114.3 -> 123.4 mm
- net test_30: track 116.3 -> 125.4 mm
- net test_19: track 151.9 -> 147.3 mm
- net test_20: track 163.9 -> 159.2 mm
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Other:
- board text added: "Rev.B1 fevereiro/2026"
- board text removed: "Rev.B1 janeiro/2026"

Commit message: ajustes para envio para produção
Routing:
- net write_data_32: track 79.2 -> 82.6 mm
- net lcd_enable: track 139.2 -> 136.0 mm
- net lcd_rs: track 147.0 -> 144.4 mm
- net test_31: track 107.2 -> 109.7 mm
- net lcd_data_0: track 138.9 -> 136.7 mm
- net test_30: track 125.4 -> 127.5 mm
- net test_7: track 89.9 -> 91.9 mm
- net test_29: track 123.4 -> 125.2 mm
- net mcu_state_error: track 110.3 -> 108.5 mm
- net console_left: track 196.5 -> 194.8 mm
- net test_6: track 110.6 -> 112.2 mm
- net console_right: track 160.0 -> 158.5 mm
- net console_back: track 161.5 -> 160.0 mm
- net lcd_data_1: track 131.1 -> 129.9 mm
- net console_ok: track 172.7 -> 171.7 mm
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