File: pcb_v2/clua/clua.kicad_sch (KiCad schematic)
At the start: 92 parts, among them J1 bus_ula_2, J10 bus_rf16_3, J2 bus_ula_1, J3 bus_rf16_1, J4 bus_rf16_2, J5 bus mem 1, J6 bus mem 2, J8 bus_mgrf_1, J9 bus_mgrf_2, SW1 RESET, U1 74LS193, U10 MC14495P, U11 IR_HIGH, U12 74LS574, U13 MC14495P, U14 RDADDR_LOW, U15 74LS138, U16 74LS86, U17 RDADDR_HIGH, U18 74LS244, U19 74LS04, U2 74HC238, U20 74LS08, U21 MC14495P, U22 WRADDR_HIGH, U23 WRADDR_LOW, U3 74LS32, U4 74LS04, U5 74LS08, U6 74LS157, U7 74LS157, U8 74LS574, U8 MC14495P, U9 IR_LOW

Commit message: experimentação com opcodes
Parts:
- removed R1: 10K, symbol Device:R
- added C24, C25, C26, C27, C28: 100nF, Capacitor_THT:C_Disc_D5.1mm_W3.2mm_P5.00mm, symbol Device:C
- added D20, D21, D22, D23: 1N4148, Diode_THT:D_DO-35_SOD27_P7.62mm_Horizontal, symbol Diode:1N4148
- added D24: CONDITION_TRUE, LED_THT:LED_D5.0mm, symbol Device:LED
- added J11: UCODE_1, edge_connector:male-edge-connector-28, symbol Connector_Generic:Conn_02x14_Top_Bottom
- added J12: UCODE_2, edge_connector:male-edge-connector-28, symbol Connector_Generic:Conn_02x14_Top_Bottom
- added J13: UCODE_3, edge_connector:male-edge-connector-28, symbol Connector_Generic:Conn_02x14_Top_Bottom
- added J14: UCODE_4, edge_connector:male-edge-connector-28, symbol Connector_Generic:Conn_02x14_Top_Bottom
- added J15: UCODE_5, edge_connector:male-edge-connector-28, symbol Connector_Generic:Conn_02x14_Top_Bottom
- added J16: UCODE_6, edge_connector:male-edge-connector-28, symbol Connector_Generic:Conn_02x14_Top_Bottom
- added J17: UCODE_7, edge_connector:male-edge-connector-28, symbol Connector_Generic:Conn_02x14_Top_Bottom
- added J18: UCODE_INT, edge_connector:male-edge-connector-28, symbol Connector_Generic:Conn_02x14_Top_Bottom
- added J7: UCODE_0, edge_connector:male-edge-connector-28, symbol Connector_Generic:Conn_02x14_Top_Bottom
- added Q1, Q2: BC548, Package_TO_SOT_THT:TO-92_Inline, symbol Transistor_BJT:BC548
- added R21, R22: 10K, Resistor_THT:R_Axial_DIN0207_L6.3mm_D2.5mm_P7.62mm_Horizontal, symbol Device:R
- added R23, R24, R25, R26, R27, R28, R29, R30, R31, R32, R33: 10K, symbol Device:R
- added R34: 1K, Resistor_THT:R_Axial_DIN0207_L6.3mm_D2.5mm_P7.62mm_Horizontal, symbol Device:R
- added U24, U25: 74LS86, symbol 74xx:74LS86
- added U26: 74LS32, symbol 74xx:74LS32
- added U27: 74LS08, symbol 74xx:74LS08
- added U28: 74LS74, symbol 74xx:74LS74
Connections:
- net +5V: now also C24.2, C25.2, C26.2, C27.2, C28.2, J11.1 (Pin_1), J11.15 (Pin_15), J12.1 (Pin_1), J12.15 (Pin_15), J13.1 (Pin_1), J13.15 (Pin_15), J14.1 (Pin_1), J14.15 (Pin_15), J15.1 (Pin_1), J15.15 (Pin_15), J16.1 (Pin_1), J16.15 (Pin_15), J17.1 (Pin_1), J17.15 (Pin_15), J18.1 (Pin_1), J18.15 (Pin_15), J7.1 (Pin_1), J7.15 (Pin_15), R34.1, U24.16 (VCC), U25.14 (VCC), U26.14 (VCC), U27.14 (VCC), U28.14 (VCC), U28.4 (~{S})
- net CARRY_FLAG: now also U24.4
- net CLOCK: now also U20.5
- net GND: now also R15.1, R16.1, R17.1, R18.1, R19.1, C24.1, C25.1, C26.1, C27.1, C28.1, J11.14 (Pin_14), J11.28 (Pin_28), J12.14 (Pin_14), J12.28 (Pin_28), J13.14 (Pin_14), J13.28 (Pin_28), J14.14 (Pin_14), J14.28 (Pin_28), J15.14 (Pin_14), J15.28 (Pin_28), J16.14 (Pin_14), J16.28 (Pin_28), J17.14 (Pin_14), J17.28 (Pin_28), J18.14 (Pin_14), J18.28 (Pin_28), J7.14 (Pin_14), J7.28 (Pin_28), Q1.1 (C), R23.1, R24.2, R25.2, R26.2, R27.2, R28.2, R29.2, R30.2, R31.2, R32.2, R33.2, U24.8 (GND), U25.7 (GND), U26.7 (GND), U27.7 (GND), U28.7 (GND); no longer R15.2, R16.2, R17.2, R18.2, R19.2, U23.3 (CA), U23.8 (CA)
- net INS_{0}: now also U26.2
- net INS_{1}: now also U26.5
- net INS_{2}: now also U26.10
- net INS_{3}: now also U26.13
- net INS_{4}: now also U24.10, U24.13, U24.2, U24.5
- net INS_{5}: now also U24.1 (A0)
- net INS_{6}: now also U24.2 (A1)
- net INS_{7}: now also U24.3 (A2)
- net NEGATIVE_FLAG: now also U24.12
- net OVERFLOW_FLAG: now also U24.9
- net RESET: now also U3.2
- net WRITE_ENABLE: now also R21.2, R22.2
- net WR_ADDR_0: now also R15.2; no longer R15.1
- net WR_ADDR_1: now also R16.2; no longer R16.1
- net WR_ADDR_2: now also R17.2; no longer R17.1
- net WR_ADDR_3: now also R18.2; no longer R18.1
- net WR_ADDR_4: now also R19.2; no longer R19.1
- net ZERO_FLAG: now also U24.1
- net fetch_cycle: now also D22.2 (A), J11.17 (Pin_17), J12.17 (Pin_17), J13.17 (Pin_17), J14.17 (Pin_17), J15.17 (Pin_17), J16.17 (Pin_17), J17.17 (Pin_17), J18.17 (Pin_17), J7.17 (Pin_17)
- net high_cycle: now also D20.2 (A), J11.19 (Pin_19), J12.19 (Pin_19), J13.19 (Pin_19), J14.19 (Pin_19), J15.19 (Pin_19), J16.19 (Pin_19), J17.19 (Pin_19), J18.19 (Pin_19), J7.19 (Pin_19)
- net low_cycle: now also D21.2 (A), J11.18 (Pin_18), J12.18 (Pin_18), J13.18 (Pin_18), J14.18 (Pin_18), J15.18 (Pin_18), J16.18 (Pin_18), J17.18 (Pin_18), J18.18 (Pin_18), J7.18 (Pin_18)
- net UC_clear_cond_reg: now reaches U3.1
- net UC_clear_cond_reg: now also J11.8 (Pin_8), J12.8 (Pin_8), J13.8 (Pin_8), J14.8 (Pin_8), J15.8 (Pin_8), J16.8 (Pin_8), J17.8 (Pin_8), J18.8 (Pin_8), J7.8 (Pin_8), R32.1
- net at U3.3: now also U4.11
- net at U22.3 (CA), U22.8 (CA): now also Q2.3 (E); no longer R20.1
- net at U4.10: now also U28.1 (~{R})
- net UC_save_cond_reg: now reaches U20.4
- net UC_save_cond_reg: now also J11.23 (Pin_23), J12.23 (Pin_23), J13.23 (Pin_23), J14.23 (Pin_23), J15.23 (Pin_23), J16.23 (Pin_23), J17.23 (Pin_23), J18.23 (Pin_23), J7.23 (Pin_23), R27.1
- net at U20.6: now also U28.3 (C)
- net UC_save_src_register renamed UC_save_src_reg
- net UC_save_src_reg: now also J11.21 (Pin_21), J12.21 (Pin_21), J13.21 (Pin_21), J14.21 (Pin_21), J15.21 (Pin_21), J16.21 (Pin_21), J17.21 (Pin_21), J18.21 (Pin_21), J7.21 (Pin_21), R25.1
- net finish_cycle: no longer names the net of U2.9 (Y6)
- net finish_cycle: now also D23.2 (A)
- net restart_fetch renamed ~{restart_fetch}
- net write_const renamed UC_write_const
- net write_enable renamed UC_write_enable
- net UC_write_enable: now also J11.27 (Pin_27), J12.27 (Pin_27), J13.27 (Pin_27), J14.27 (Pin_27), J15.27 (Pin_27), J16.27 (Pin_27), J17.27 (Pin_27), J18.27 (Pin_27), J7.27 (Pin_27), R31.1
- net ~{inhibit_write} renamed condition_true
- net condition_true: now also U28.6 (~{Q})
- new net: D20.1 (K), D21.1 (K), D22.1 (K), R23.2, U24.6 (E3)
- new net: U24.8, U26.9
- new net: U27.10, U27.6
- new net: U27.8, U28.2 (D)
- new net: U27.3, U27.9
- new net: U24.6, U26.4
- new net: U26.6, U27.2
- new net: Q2.1 (C), R20.1
- new net: U26.8, U27.4
- new net: U26.11, U27.5
- new net: Q1.2 (B), R21.1
- new net: Q1.3 (E), U23.3 (CA), U23.8 (CA)
- new net: U24.3, U26.1
- new net: U24.11, U26.12
- new net: D24.2 (A), R34.2
- new net: Q2.2 (B), R22.1
- new net: U26.3, U27.1
- new net UC_int_cycle: J11.20 (Pin_20), J12.20 (Pin_20), J13.20 (Pin_20), J14.20 (Pin_20), J15.20 (Pin_20), J16.20 (Pin_20), J17.20 (Pin_20), J18.20 (Pin_20), J7.20 (Pin_20), R24.1
- new net UC_pcia_swap: J11.25 (Pin_25), J12.25 (Pin_25), J13.25 (Pin_25), J14.25 (Pin_25), J15.25 (Pin_25), J16.25 (Pin_25), J17.25 (Pin_25), J18.25 (Pin_25), J7.25 (Pin_25), R29.1
- new net UC_pclr_swap: J11.24 (Pin_24), J12.24 (Pin_24), J13.24 (Pin_24), J14.24 (Pin_24), J15.24 (Pin_24), J16.24 (Pin_24), J17.24 (Pin_24), J18.24 (Pin_24), J7.24 (Pin_24), R28.1
- new net UC_restart_cycle: D23.1 (K), J11.22 (Pin_22), J12.22 (Pin_22), J13.22 (Pin_22), J14.22 (Pin_22), J15.22 (Pin_22), J16.22 (Pin_22), J17.22 (Pin_22), J18.22 (Pin_22), J7.22 (Pin_22), R26.1
- new net UC_ula_enable: J11.9 (Pin_9), J12.9 (Pin_9), J13.9 (Pin_9), J14.9 (Pin_9), J15.9 (Pin_9), J16.9 (Pin_9), J17.9 (Pin_9), J18.9 (Pin_9), J7.9 (Pin_9), R33.1
- new net UC_write_address: J11.26 (Pin_26), J12.26 (Pin_26), J13.26 (Pin_26), J14.26 (Pin_26), J15.26 (Pin_26), J16.26 (Pin_26), J17.26 (Pin_26), J18.26 (Pin_26), J7.26 (Pin_26), R30.1
- new net select_opcode_0: J7.16 (Pin_16), U24.15 (Y0)
- new net select_opcode_1: J11.16 (Pin_16), U24.14 (Y1)
- new net select_opcode_2: J12.16 (Pin_16), U24.13 (Y2)
- new net select_opcode_3: J13.16 (Pin_16), U24.12 (Y3)
- new net select_opcode_4: J14.16 (Pin_16), U24.11 (Y4)
- new net select_opcode_5: J15.16 (Pin_16), U24.10 (Y5)
- new net select_opcode_6: J16.16 (Pin_16), U24.9 (Y6)
- new net select_opcode_7: J17.16 (Pin_16), U24.7 (Y7)
- new net select_opcode_int: J18.16 (Pin_16)
- new net ~{UC_int_cycle}: U24.4 (~{E1}), U24.5 (~{E2})
- new net ~{condition_true}: D24.1 (K), U28.5 (Q)
- no-connect marks 56 -> 146
Other:
- note removed: "CORRIGIR MEMA! Ordem dos sinais está errada"
- moved on the sheet: C10, C12, C13, C15, C18, C6, C7, C8, D1, D10, D11, D12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

Commit message: continuando com a implementação da lógica de controle; ROM de ucode expandida para 17 bits
Parts:
- added C19, C29, C30: 100nF, Capacitor_THT:C_Disc_D5.1mm_W3.2mm_P5.00mm, symbol Device:C
- added R35: 10K, symbol Device:R
- added unit 6 of U19
- added unit 4 of U19
- added unit 2 of U19
- added unit 5 of U19
- added unit 7 of U19
- added unit 1 of U19
- added U29: 74LS74, symbol 74xx:74LS74
- added U30: 74LS138, symbol 74xx:74LS138
Connections:
- net FLAG_INTMASK is gone; now on net INT_MASK_FLAG: J1.1 (Pin_1)
- net halt is gone; now on net GND: U2.4 (~{E1}), U2.5 (~{E2})
- net reset is gone; now on net RESET: U1.14 (CLR)
- net +5V: now also R24.2, R25.2, R26.2, R27.2, R28.2, R29.2, R30.2, R31.2, R32.2, R33.2, U28.10 (~{S}), C19.2, C29.2, C30.2, R35.2, U19.14 (VCC), U29.14 (VCC), U29.2 (D), U29.4 (~{S}), U30.16 (VCC), U30.6 (E3); no longer U2.6 (E3)
- net GND: now also C19.1, C29.1, C30.1, U19.7 (GND), U29.11 (C), U29.12 (D), U29.7 (GND), U30.8 (GND); no longer R24.2, R25.2, R26.2, R27.2, R28.2, R29.2, R30.2, R31.2, R32.2, R33.2
- net INS_{0}: now also U30.1 (A0)
- net INS_{1}: now also U30.2 (A1)
- net INS_{2}: now also U30.3 (A2)
- net UC_restart_cycle: now also U19.9; no longer J11.22 (Pin_22), J12.22 (Pin_22), J13.22 (Pin_22), J14.22 (Pin_22), J15.22 (Pin_22), J16.22 (Pin_22), J17.22 (Pin_22), J18.22 (Pin_22), J7.22 (Pin_22), R26.1
- net UC_save_src_reg: no longer J11.21 (Pin_21), J12.21 (Pin_21), J13.21 (Pin_21), J14.21 (Pin_21), J15.21 (Pin_21), J16.21 (Pin_21), J17.21 (Pin_21), J18.21 (Pin_21), J7.21 (Pin_21), R25.1
- net UC_write_enable: no longer J11.27 (Pin_27), J12.27 (Pin_27), J13.27 (Pin_27), J14.27 (Pin_27), J15.27 (Pin_27), J16.27 (Pin_27), J17.27 (Pin_27), J18.27 (Pin_27), J7.27 (Pin_27), R31.1
- net select_opcode_int: now also U24.4 (~{E1}), U24.5 (~{E2}), U28.9 (Q)
- net ~{UC_int_cycle}: now also R24.1; no longer U24.4 (~{E1}), U24.5 (~{E2})
- net at U28.11 (C): now also U4.12
- net int_pending: now reaches U28.12 (D)
- net int_pending: now also U29.5 (Q)
- net ~{UC_restart_cycle}: now reaches U28.13 (~{R})
- net ~{UC_restart_cycle}: now also J11.13 (Pin_13), J12.13 (Pin_13), J13.13 (Pin_13), J14.13 (Pin_13), J15.13 (Pin_13), J16.13 (Pin_13), J17.13 (Pin_13), J18.13 (Pin_13), J7.13 (Pin_13), R26.1
- net ~{UC_save_src_reg}: now reaches J17.12 (Pin_12)
- net ~{UC_save_src_reg}: now also J11.12 (Pin_12), J12.12 (Pin_12), J13.12 (Pin_12), J14.12 (Pin_12), J15.12 (Pin_12), J16.12 (Pin_12), J18.12 (Pin_12), J7.12 (Pin_12), R25.1
- net ~{UC_save_cond_reg}: now reaches J17.4 (Pin_4)
- net ~{UC_save_cond_reg}: now also J11.4 (Pin_4), J12.4 (Pin_4), J13.4 (Pin_4), J14.4 (Pin_4), J15.4 (Pin_4), J16.4 (Pin_4), J18.4 (Pin_4), J7.4 (Pin_4), R27.1, U19.1
- net ~{UC_clear_cond_reg}: now reaches J17.5 (Pin_5)
- net ~{UC_clear_cond_reg}: now also J11.5 (Pin_5), J12.5 (Pin_5), J13.5 (Pin_5), J14.5 (Pin_5), J15.5 (Pin_5), J16.5 (Pin_5), J18.5 (Pin_5), J7.5 (Pin_5), R32.1, U19.3
- net ~{UC_ula_enable}: now reaches J17.6 (Pin_6)
- net ~{UC_ula_enable}: now also J11.6 (Pin_6), J12.6 (Pin_6), J13.6 (Pin_6), J14.6 (Pin_6), J15.6 (Pin_6), J16.6 (Pin_6), J18.6 (Pin_6), J7.6 (Pin_6), R33.1
- net ~{UC_pclr_swap}: now reaches J17.7 (Pin_7)
- net ~{UC_pclr_swap}: now also J11.7 (Pin_7), J12.7 (Pin_7), J13.7 (Pin_7), J14.7 (Pin_7), J15.7 (Pin_7), J16.7 (Pin_7), J18.7 (Pin_7), J7.7 (Pin_7), R28.1
- net ~{UC_int_ready}: now reaches U4.13
- net ~{UC_int_ready}: now also J11.22 (Pin_22), J12.22 (Pin_22), J13.22 (Pin_22), J14.22 (Pin_22), J15.22 (Pin_22), J16.22 (Pin_22), J17.22 (Pin_22), J18.22 (Pin_22), J7.22 (Pin_22)
- net at U20.11: now also U29.3 (C)
- net INT_REQUEST: now reaches U20.12
- net INT_MASK_FLAG: now reaches U20.13
- net INT_MASK_FLAG: now also U29.9 (Q)
- removed net UC_clear_cond_reg: J11.8 (Pin_8), J12.8 (Pin_8), J13.8 (Pin_8), J14.8 (Pin_8), J15.8 (Pin_8), J16.8 (Pin_8), J17.8 (Pin_8), J18.8 (Pin_8), J7.8 (Pin_8), R32.1, U3.1
- removed net UC_int_cycle: J11.20 (Pin_20), J12.20 (Pin_20), J13.20 (Pin_20), J14.20 (Pin_20), J15.20 (Pin_20), J16.20 (Pin_20), J17.20 (Pin_20), J18.20 (Pin_20), J7.20 (Pin_20), R24.1
- removed net UC_pcia_swap: J11.25 (Pin_25), J12.25 (Pin_25), J13.25 (Pin_25), J14.25 (Pin_25), J15.25 (Pin_25), J16.25 (Pin_25), J17.25 (Pin_25), J18.25 (Pin_25), J7.25 (Pin_25), R29.1
- removed net UC_pclr_swap: J11.24 (Pin_24), J12.24 (Pin_24), J13.24 (Pin_24), J14.24 (Pin_24), J15.24 (Pin_24), J16.24 (Pin_24), J17.24 (Pin_24), J18.24 (Pin_24), J7.24 (Pin_24), R28.1
- net UC_save_cond_reg renamed ~{UC_pcia_swap}
- net ~{UC_pcia_swap}: now also R29.1; no longer R27.1, U20.4
- removed net UC_ula_enable: J11.9 (Pin_9), J12.9 (Pin_9), J13.9 (Pin_9), J14.9 (Pin_9), J15.9 (Pin_9), J16.9 (Pin_9), J17.9 (Pin_9), J18.9 (Pin_9), J7.9 (Pin_9), R33.1
- net UC_write_address renamed ~{UC_write_address}
- net ~{restart_fetch}: no longer names the net of U1.11 (~{LOAD})
- net ~{restart_fetch}: now also U19.8
- new net: U19.4, U3.1
- new net: U19.2, U20.4
- new net ~{UC_break}: U30.10 (O5)
- new net ~{UC_clear_interrupt_mask}: U29.13 (~{R}), U30.12 (O3)
- new net ~{UC_clear_pending_int}: U29.1 (~{R}), U30.14 (O1)
- new net ~{UC_extended_opcode}: R35.1, U30.4 (E1), U30.5 (E2)
- new net ~{UC_halt}: U2.6 (E3), U30.11 (O4)
- new net ~{UC_set_interrupt_mask}: U29.10 (~{S}), U30.13 (O2)
- new net ~{UC_write_enable}: J11.27 (Pin_27), J12.27 (Pin_27), J13.27 (Pin_27), J14.27 (Pin_27), J15.27 (Pin_27), J16.27 (Pin_27), J17.27 (Pin_27), J18.27 (Pin_27), J7.27 (Pin_27), R31.1
- no-connect marks 146 -> 150
Other:
- moved on the sheet: C10, C16, C20, C25, C26, C27, C28, C3, C4, C6, C7, C8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

Commit message: .
Parts:
- removed R29: 10K, symbol Device:R
- renumbered C8 to C31, C24 to C32, C10 to C9, U25 to U24, U8 to U31, U24 to U32
Connections:
- net UC_save_src_reg is gone; now on an unnamed net: U5.12
- net +5V: no longer U30.6 (E3)
- net CLOCK: now also U30.6 (E3)
- net fetch_cycle: now also J11.16 (Pin_16), J12.16 (Pin_16), J13.16 (Pin_16), J14.16 (Pin_16), J15.16 (Pin_16), J16.16 (Pin_16), J17.16 (Pin_16), J18.16 (Pin_16), J7.16 (Pin_16); no longer J11.17 (Pin_17), J12.17 (Pin_17), J13.17 (Pin_17), J14.17 (Pin_17), J15.17 (Pin_17), J16.17 (Pin_17), J17.17 (Pin_17), J18.17 (Pin_17), J7.17 (Pin_17)
- net high_cycle: now also J11.17 (Pin_17), J12.17 (Pin_17), J13.17 (Pin_17), J14.17 (Pin_17), J15.17 (Pin_17), J16.17 (Pin_17), J17.17 (Pin_17), J18.17 (Pin_17), J7.17 (Pin_17); no longer J11.19 (Pin_19), J12.19 (Pin_19), J13.19 (Pin_19), J14.19 (Pin_19), J15.19 (Pin_19), J16.19 (Pin_19), J17.19 (Pin_19), J18.19 (Pin_19), J7.19 (Pin_19)
- net select_opcode_0: now also J7.19 (Pin_19); no longer J7.16 (Pin_16)
- net select_opcode_1: now also J11.19 (Pin_19); no longer J11.16 (Pin_16)
- net select_opcode_2: now also J12.19 (Pin_19); no longer J12.16 (Pin_16)
- net select_opcode_3: now also J13.19 (Pin_19); no longer J13.16 (Pin_16)
- net select_opcode_4: now also J14.19 (Pin_19); no longer J14.16 (Pin_16)
- net select_opcode_5: now also J15.19 (Pin_19); no longer J15.16 (Pin_16)
- net select_opcode_6: now also J16.19 (Pin_19); no longer J16.16 (Pin_16)
- net select_opcode_7: now also J17.19 (Pin_19); no longer J17.16 (Pin_16)
- net select_opcode_int: now also J18.19 (Pin_19); no longer J18.16 (Pin_16)
- net ~{UC_clear_cond_reg}: now also J11.26 (Pin_26), J12.26 (Pin_26), J13.26 (Pin_26), J14.26 (Pin_26), J15.26 (Pin_26), J16.26 (Pin_26), J17.26 (Pin_26), J18.26 (Pin_26), J7.26 (Pin_26); no longer J11.5 (Pin_5), J12.5 (Pin_5), J13.5 (Pin_5), J14.5 (Pin_5), J15.5 (Pin_5), J16.5 (Pin_5), J17.5 (Pin_5), J18.5 (Pin_5), J7.5 (Pin_5)
- net ~{UC_extended_opcode}: now also J11.6 (Pin_6), J12.6 (Pin_6), J13.6 (Pin_6), J14.6 (Pin_6), J15.6 (Pin_6), J16.6 (Pin_6), J17.6 (Pin_6), J18.6 (Pin_6), J7.6 (Pin_6)
- net ~{UC_pclr_swap}: no longer J11.7 (Pin_7), J12.7 (Pin_7), J13.7 (Pin_7), J14.7 (Pin_7), J15.7 (Pin_7), J16.7 (Pin_7), J17.7 (Pin_7), J18.7 (Pin_7), J7.7 (Pin_7)
- net ~{UC_restart_cycle}: now also J11.12 (Pin_12), J12.12 (Pin_12), J13.12 (Pin_12), J14.12 (Pin_12), J15.12 (Pin_12), J16.12 (Pin_12), J17.12 (Pin_12), J18.12 (Pin_12), J7.12 (Pin_12); no longer J11.13 (Pin_13), J12.13 (Pin_13), J13.13 (Pin_13), J14.13 (Pin_13), J15.13 (Pin_13), J16.13 (Pin_13), J17.13 (Pin_13), J18.13 (Pin_13), J7.13 (Pin_13)
- net ~{UC_save_cond_reg}: now also J11.20 (Pin_20), J12.20 (Pin_20), J13.20 (Pin_20), J14.20 (Pin_20), J15.20 (Pin_20), J16.20 (Pin_20), J17.20 (Pin_20), J18.20 (Pin_20), J7.20 (Pin_20); no longer J11.4 (Pin_4), J12.4 (Pin_4), J13.4 (Pin_4), J14.4 (Pin_4), J15.4 (Pin_4), J16.4 (Pin_4), J17.4 (Pin_4), J18.4 (Pin_4), J7.4 (Pin_4)
- net ~{UC_save_src_reg}: now also J11.25 (Pin_25), J12.25 (Pin_25), J13.25 (Pin_25), J14.25 (Pin_25), J15.25 (Pin_25), J16.25 (Pin_25), J17.25 (Pin_25), J18.25 (Pin_25), J7.25 (Pin_25), U19.11; no longer J11.12 (Pin_12), J12.12 (Pin_12), J13.12 (Pin_12), J14.12 (Pin_12), J15.12 (Pin_12), J16.12 (Pin_12), J17.12 (Pin_12), J18.12 (Pin_12), J7.12 (Pin_12)
- net ~{UC_ula_enable}: now also J11.8 (Pin_8), J12.8 (Pin_8), J13.8 (Pin_8), J14.8 (Pin_8), J15.8 (Pin_8), J16.8 (Pin_8), J17.8 (Pin_8), J18.8 (Pin_8), J7.8 (Pin_8); no longer J11.6 (Pin_6), J12.6 (Pin_6), J13.6 (Pin_6), J14.6 (Pin_6), J15.6 (Pin_6), J16.6 (Pin_6), J17.6 (Pin_6), J18.6 (Pin_6), J7.6 (Pin_6)
- net ~{UC_write_address}: now also J11.13 (Pin_13), J12.13 (Pin_13), J13.13 (Pin_13), J14.13 (Pin_13), J15.13 (Pin_13), J16.13 (Pin_13), J17.13 (Pin_13), J18.13 (Pin_13), J7.13 (Pin_13); no longer J11.26 (Pin_26), J12.26 (Pin_26), J13.26 (Pin_26), J14.26 (Pin_26), J15.26 (Pin_26), J16.26 (Pin_26), J17.26 (Pin_26), J18.26 (Pin_26), J7.26 (Pin_26)
- net ~{UC_write_enable}: now also J11.21 (Pin_21), J12.21 (Pin_21), J13.21 (Pin_21), J14.21 (Pin_21), J15.21 (Pin_21), J16.21 (Pin_21), J17.21 (Pin_21), J18.21 (Pin_21), J7.21 (Pin_21); no longer J11.27 (Pin_27), J12.27 (Pin_27), J13.27 (Pin_27), J14.27 (Pin_27), J15.27 (Pin_27), J16.27 (Pin_27), J17.27 (Pin_27), J18.27 (Pin_27), J7.27 (Pin_27)
- no-connect marks 150 -> 173
Other:
- moved on the sheet: C30, C9, D1, J1, J11, J13, J14, J16, J2, R1, R30, R31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

Commit message: revisando o ERC
Parts:
- removed R2, R3, R4: 10K, symbol Device:R
- removed U15: 74LS138, symbol 74xx:74LS138
- removed unit 4 of U16
- removed unit 3 of U16
- removed unit 2 of U16
- removed unit 6 of U19
- removed unit 3 of U19
- removed unit 3 of U20
- removed unit 4 of U27
- removed unit 2 of U3
- removed unit 3 of U3
- removed unit 4 of U3
- removed unit 4 of U4
- removed unit 3 of U4
- removed unit 1 of U5
- added C11: 0.33uF, Capacitor_THT:CP_Radial_D5.0mm_P2.50mm, symbol Device:C_Polarized
- added C14: 0.1uF, Capacitor_THT:CP_Radial_D5.0mm_P2.50mm, symbol Device:C_Polarized
- added C25: 100nF, Capacitor_THT:C_Disc_D5.1mm_W3.2mm_P5.00mm, symbol Device:C
- added D25, D26, D27, D28, D29, D30, D31: 1N4148, Diode_THT:D_DO-35_SOD27_P7.62mm_Horizontal, symbol Diode:1N4148
- added D32: 1N4001, Diode_THT:D_DO-41_SOD81_P10.16mm_Horizontal, symbol Diode:1N4001
- added J19: 9V 1A, symbol Connector_Generic:Conn_01x02
- added J20: VOLTMETER, symbol Connector_Generic:Conn_01x02
- added J21: AMPMETER, symbol Connector_Generic:Conn_01x02
- added R29, R36, R37, R38, R39, R40, R41, R42, R43, R44, R45, R46, R47, R48, R49, R50, R51, R52: 10K, symbol Device:R
- added U15: 74LS04, symbol 74xx:74LS04
- added U25: 74LS125, symbol 74xx:74LS125
- added U33: 74LS32, symbol 74xx:74LS32
- added U34: LM7805, Package_TO_SOT_THT:TO-220-3_Vertical, symbol Regulator_Linear:LM7805_TO220
Connections:
- net ~{write_address} is gone; now on net ~{UC_write_address}: U18.1 (OEa), U18.19 (OEb)
- net +5V: now also C25.2, J20.2 (Pin_2), J21.2 (Pin_2), R29.2, R36.2, R37.2, R38.2, R39.2, R40.2, R41.2, R42.2, R43.2, R44.2, R45.2, R46.2, R47.2, R48.2, R49.2, R50.2, R51.2, U15.14 (VCC), U25.14 (VCC)
- net ADDR_{0}: now also R51.1, U25.3
- net ADDR_{10}: now also R41.1
- net ADDR_{11}: now also R40.1
- net ADDR_{12}: now also R39.1
- net ADDR_{13}: now also R38.1
- net ADDR_{14}: now also R37.1
- net ADDR_{15}: now also R36.1
- net ADDR_{1}: now also R50.1, U25.6
- net ADDR_{2}: now also R49.1
- net ADDR_{3}: now also R48.1
- net ADDR_{4}: now also R47.1
- net ADDR_{5}: now also R46.1
- net ADDR_{6}: now also R45.1
- net ADDR_{7}: now also R44.1
- net ADDR_{8}: now also R43.1
- net ADDR_{9}: now also R42.1
- net GND: now also C11.2, C14.2, C25.1, J19.1 (Pin_1), J20.1 (Pin_1), R52.2, U15.7 (GND), U25.7 (GND), U34.2 (GND)
- net UC_read_mem_const: now also D3.2 (A), D4.2 (A), D5.2 (A), D6.2 (A), D7.2 (A), D26.1 (K), D27.1 (K)
- net UC_read_mem_pc: now also D10.2 (A), D11.2 (A), D12.2 (A), D8.2 (A), D9.2 (A), D25.1 (K)
- net UC_write_enable: now also U5.4, D30.1 (K), D31.1 (K)
- net fetch_cycle: now also D25.2 (A)
- net high_cycle: now also U33.2
- net reset_high_cycle: now also D27.2 (A), D29.2 (A), D31.2 (A), U33.1
- net reset_low_cycle: now also D26.2 (A), D28.2 (A), D30.2 (A)
- net ~{UC_pcia_swap}: now also R28.1
- net ~{UC_pclr_swap}: now also U30.9 (O6); no longer R28.1
- net wr_addr_pc: now reaches D16.2 (A), D17.2 (A), D18.2 (A), D19.2 (A), U20.2
- net ~{UC_read_addr_src_reg}: now reaches J17.27 (Pin_27)
- net ~{UC_read_addr_src_reg}: now also J11.27 (Pin_27), J12.27 (Pin_27), J13.27 (Pin_27), J14.27 (Pin_27), J15.27 (Pin_27), J16.27 (Pin_27), J18.27 (Pin_27), J7.27 (Pin_27), R29.1
- net ~{rd_addr_output_register} renamed ~{UC_rd_addr_src_reg}
- new net: C14.1, J21.1 (Pin_1), U34.3 (VO)
- new net: C11.1, D32.1 (K), U34.1 (VI)
- new net: U25.2, U33.3
- new net +9V: D32.2 (A), J19.2 (Pin_2)
- new net UC_const_boot_addr: D28.1 (K), D29.1 (K), R52.1, U25.5
- new net ~{UC_read_mem_const}: U25.1, U25.4
- no-connect marks 173 -> 136
Other:
- moved on the sheet: C12, C18, C30, D10, D11, D12, D24, D3, D4, D5, D6, D7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
