File: pcb_v2/clua/clua.kicad_pcb (KiCad board)
At the start: 2 copper layers, 109 parts, among them J1 bus clu 1, J11 UCODE_1, J12 UCODE_2, J13 UCODE_3, J14 UCODE_4, J15 UCODE_5, J16 UCODE_6, J17 UCODE_7, J18 UCODE_INT, J2 bus clu 2, J3 bus clu 3, J7 UCODE_0, U1 74LS193, U10 MC14495P, U11 IR_HIGH, U12 74LS574, U16 74LS86, U18 74LS244, U19 74LS04, U2 74HC238, U20 74LS08, U24 74LS86, U25 74LS125, U26 74LS32, U27 74LS08, U28 74LS74, U29 74LS74, U30 74LS138, U31 MC14495P, U32 74HC238, U4 74LS02, U6 74LS157, U7 74LS157, U8 74LS574, U9 IR_LOW

Commit message: refazendo os pcbs para caber em folha A4
Parts:
- removed R1, R10, R3, R4, R9: 10K, Resistor_THT:R_Axial_DIN0207_L6.3mm_D2.5mm_P7.62mm_Horizontal
- J1: value bus clu 1 -> sysbus_1
- J2: value bus clu 2 -> sysbus_2
- J3: value bus clu 3 -> sysbus_3
- U16, U19, U20, U24, U25, U26, U27, U28, U29: footprint Package_DIP:DIP-14_W10.16mm -> Package_DIP:DIP-14_W7.62mm
- U2: footprint Package_DIP:DIP-20_W7.62mm -> Package_DIP:DIP-16_W7.62mm
- U8: footprint Package_DIP:DIP-16_W7.62mm -> Package_DIP:DIP-20_W7.62mm
- moved C31 385.0 mm to (57.9, 182.2)
- moved C10 375.2 mm to (47.1, 182.2)
- moved R35 361.3 mm to (55.2, 35.6), turned to 90 degrees
- moved R27 355.7 mm to (51.4, 35.6), turned to 90 degrees
- moved R31 353.9 mm to (59.1, 35.6), turned to 90 degrees
- moved R33 348.3 mm to (66.7, 35.6), turned to 90 degrees
- moved C32 342.6 mm to (102.9, 186.1), turned to -90 degrees
- moved R24 341.5 mm to (62.9, 35.6), turned to 90 degrees
- moved C2 339.5 mm to (102.9, 200.1), turned to -90 degrees
- moved R28 338.5 mm to (70.5, 35.6), turned to 90 degrees
- moved R32 336.2 mm to (78.1, 35.6), turned to 90 degrees
- moved C29 331.9 mm to (102.3, 137.8)
- moved R25 331.5 mm to (74.3, 35.6), turned to 90 degrees
- moved R13 329.2 mm to (87.0, 224.8), turned to 90 degrees
- moved C28 328.1 mm to (134.6, 200.1), turned to -90 degrees
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Connections:
- D15 pad 2: Net-(D15-A) -> wr_addr_pc
- D3 pad 1: rd_addr_lsb -> RD_ADDR_0
- D8 pad 1: rd_addr_lsb -> RD_ADDR_0
- U12 pad 19: rd_addr_lsb -> RD_ADDR_0
- U16 pad 1: high_cycle -> +5V
- U16 pad 2: rd_addr_lsb -> +5V
- U16 pad 3: RD_ADDR_0 -> unconnected-(U16-Pad3)
- U20 pad 1: high_cycle -> +5V
- U20 pad 2: wr_addr_pc -> +5V
- U20 pad 3: Net-(D15-A) -> unconnected-(U20-Pad3)
Routing:
- net +5V: track 0.00 -> 625.9 mm
- net ~{UC_extended_opcode}: track 0.00 -> 151.5 mm
- net ~{UC_save_cond_reg}: track 0.00 -> 148.8 mm
- net ~{UC_write_address}: track 0.00 -> 148.4 mm
- net ~{UC_ula_enable}: track 0.00 -> 145.1 mm
- net ~{UC_restart_cycle}: track 0.00 -> 144.1 mm
- net ~{UC_write_enable}: track 0.00 -> 143.3 mm
- net ~{UC_int_ready}: track 0.00 -> 141.7 mm
- net ~{UC_read_addr_src_reg}: track 0.00 -> 140.7 mm
- net ~{UC_save_src_reg}: track 0.00 -> 139.0 mm
- net ~{UC_pcia_swap}: track 0.00 -> 138.5 mm
- net ~{UC_clear_cond_reg}: track 0.00 -> 138.5 mm
- net low_cycle: track 0.00 -> 130.3 mm
- net high_cycle: track 0.00 -> 130.3 mm
- net fetch_clock: track 0.00 -> 130.3 mm
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- added copper zone on B.Cu, net GND
- added copper zone on F.Cu, net GND
Other:
- board outline added: 122 x 210 mm

Commit message: inicio de layout da CL
Parts:
- moved J7 136.1 mm to (31.1, 35.6), turned to 0 degrees
- moved C2 127.5 mm to (43.9, 87.0), turned to 0 degrees
- moved C32 123.9 mm to (28.6, 87.0), turned to 0 degrees
- moved U2 121.3 mm to (41.3, 90.8), turned to 0 degrees
- moved J11 119.6 mm to (43.8, 35.6), turned to 0 degrees
- moved U32 118.0 mm to (26.0, 90.8), turned to 0 degrees
- moved R27 107.0 mm to (157.5, 49.5), turned to 0 degrees
- moved J12 104.3 mm to (56.5, 35.6), turned to 0 degrees
- moved R24 96.3 mm to (157.5, 53.3), turned to 0 degrees
- moved R35 92.2 mm to (146.7, 47.6), turned to 0 degrees
- moved J13 90.7 mm to (69.2, 35.6), turned to 0 degrees
- moved R28 89.6 mm to (157.5, 57.1), turned to 0 degrees
- moved R31 89.1 mm to (146.7, 51.4), turned to 0 degrees
- moved U27 88.2 mm to (56.5, 90.8), turned to 0 degrees
- moved C27 84.9 mm to (59.1, 87.0), turned to 0 degrees
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Routing:
- net +5V: track 625.9 -> 0.00 mm
- net ~{UC_extended_opcode}: track 151.5 -> 0.00 mm
- net ~{UC_save_cond_reg}: track 148.8 -> 0.00 mm
- net ~{UC_write_address}: track 148.4 -> 0.00 mm
- net ~{UC_ula_enable}: track 145.1 -> 0.00 mm
- net ~{UC_restart_cycle}: track 144.1 -> 0.00 mm
- net ~{UC_write_enable}: track 143.3 -> 0.00 mm
- net ~{UC_int_ready}: track 141.7 -> 0.00 mm
- net ~{UC_read_addr_src_reg}: track 140.7 -> 0.00 mm
- net ~{UC_save_src_reg}: track 139.0 -> 0.00 mm
- net ~{UC_pcia_swap}: track 138.5 -> 0.00 mm
- net ~{UC_clear_cond_reg}: track 138.5 -> 0.00 mm
- net low_cycle: track 130.3 -> 0.00 mm
- net high_cycle: track 130.3 -> 0.00 mm
- net fetch_clock: track 130.3 -> 0.00 mm
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Other:
- board size 122 x 210 mm -> 160.7 x 210 mm

Commit message: layout avançando
Parts:
- moved D19 78.1 mm to (140.3, 147.3), turned to 180 degrees
- moved D18 75.1 mm to (140.3, 144.1), turned to 180 degrees
- moved D17 72.3 mm to (140.3, 141.0), turned to 180 degrees
- moved D16 69.6 mm to (140.3, 137.8), turned to 180 degrees
- moved D15 67.2 mm to (140.3, 134.6), turned to 180 degrees
- moved U29 51.8 mm to (56.5, 177.8)
- moved U6 51.8 mm to (71.7, 177.8)
- moved C29 51.8 mm to (59.1, 174.0)
- moved C6 51.8 mm to (74.4, 174.0)
- moved R2 35.6 mm to (157.5, 39.4)
- moved D26 35.6 mm to (146.7, 39.4)
- moved D30 35.6 mm to (146.7, 42.5)
- moved D20 23.2 mm to (26.0, 121.3), turned to 0 degrees
- moved D21 19.7 mm to (26.0, 118.1), turned to 0 degrees
- moved D22 16.7 mm to (26.0, 114.9), turned to 0 degrees
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Routing:
- net +5V: track 0.00 -> 848.9 mm
- net low_cycle: track 0.00 -> 410.6 mm, vias 0 -> 6
- net high_cycle: track 0.00 -> 335.9 mm, vias 0 -> 5
- net fetch_clock: track 0.00 -> 330.9 mm, vias 0 -> 3
- net ~{UC_restart_cycle}: track 0.00 -> 301.2 mm, vias 0 -> 2
- net select_opcode_int: track 0.00 -> 284.5 mm, vias 0 -> 1
- net ~{UC_pcia_swap}: track 0.00 -> 278.1 mm, vias 0 -> 3
- net ~{UC_extended_opcode}: track 0.00 -> 245.1 mm, vias 0 -> 2
- net ~{UC_write_address}: track 0.00 -> 209.2 mm, vias 0 -> 2
- net ~{UC_read_addr_src_reg}: track 0.00 -> 208.9 mm, vias 0 -> 2
- net ~{UC_write_enable}: track 0.00 -> 203.2 mm, vias 0 -> 2
- net ~{UC_int_ready}: track 0.00 -> 189.5 mm, vias 0 -> 2
- net fetch_cycle: track 0.00 -> 177.6 mm, vias 0 -> 3
- net ~{UC_ula_enable}: track 0.00 -> 176.7 mm, vias 0 -> 1
- net Net-(U29A-C): track 0.00 -> 169.0 mm, vias 0 -> 2
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
Commit message: correções no esquemático e reiniciando o pcb
Parts:
- removed D15, D26, D3, D30, D8: 1N4148, Diode_THT:D_DO-35_SOD27_P7.62mm_Horizontal
- added C3: 100nF, Capacitor_THT:C_Disc_D5.1mm_W3.2mm_P5.00mm, F.Cu at (85.2, 173.4)
- added C5: 100nF, Capacitor_THT:C_Disc_D5.1mm_W3.2mm_P5.00mm, F.Cu at (101.7, 173.4)
- added J4: UCODE_RESET, edge_connector:male-edge-connector-28, F.Cu at (145.4, 35.6)
- added SW1: SW_DIP_x04, Button_Switch_THT:SW_DIP_SPSTx04_Slide_6.7x11.72mm_W7.62mm_P2.54mm_LowProfile, F.Cu at (27.9, 192.4)
- added SW3: SW_DIP_x04, Button_Switch_THT:SW_DIP_SPSTx04_Slide_6.7x11.72mm_W7.62mm_P2.54mm_LowProfile, F.Cu at (55.9, 192.4)
- added SW6: SW_DIP_x04, Button_Switch_THT:SW_DIP_SPSTx04_Slide_6.7x11.72mm_W7.62mm_P2.54mm_LowProfile, F.Cu at (41.9, 192.4)
- added U3: 74HC04, Package_DIP:DIP-14_W7.62mm, F.Cu at (82.6, 177.2)
- added U5: 74LS32, Package_DIP:DIP-14_W7.62mm, F.Cu at (99.1, 177.2)
- D24: value CONDITION_TRUE -> TRUE
- J1: value sysbus_1 -> bus clu 1
- J2: value sysbus_2 -> bus clu 2
- J3: value sysbus_3 -> bus clu 3
- moved D4 142.7 mm to (36.8, 171.4)
- moved D5 142.7 mm to (33.7, 171.4)
- moved D6 142.7 mm to (30.5, 171.4)
- moved D7 142.7 mm to (27.3, 171.4)
- moved C1 126.7 mm to (28.7, 87.0)
- moved U1 126.7 mm to (26.0, 90.8)
- moved C28 104.4 mm to (78.2, 87.0)
- moved U28 104.4 mm to (75.6, 90.8)
- moved D19 102.0 mm to (41.3, 171.4), turned to -90 degrees
- moved D18 99.7 mm to (44.5, 171.4), turned to -90 degrees
- moved D17 97.6 mm to (47.6, 171.4), turned to -90 degrees
- moved D16 95.7 mm to (50.8, 171.4), turned to -90 degrees
- moved C29 87.0 mm to (61.7, 87.0)
- moved U29 87.0 mm to (59.1, 90.8)
- moved C24 71.5 mm to (61.7, 128.3)
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Connections:
- D10 pad 2: fetch_cycle -> Net-(D10-A)
- D11 pad 2: fetch_cycle -> Net-(D11-A)
- D12 pad 2: fetch_cycle -> Net-(D12-A)
- D16 pad 2: wr_addr_pc -> Net-(D16-A)
- D17 pad 2: wr_addr_pc -> Net-(D17-A)
- D18 pad 2: wr_addr_pc -> Net-(D18-A)
- D19 pad 2: wr_addr_pc -> Net-(D19-A)
- D4 pad 2: UC_read_mem_const -> Net-(D4-A)
- D5 pad 2: UC_read_mem_const -> Net-(D5-A)
- D6 pad 2: UC_read_mem_const -> Net-(D6-A)
- D7 pad 2: UC_read_mem_const -> Net-(D7-A)
- D9 pad 2: fetch_cycle -> Net-(D9-A)
- J11 pad 13: ~{UC_write_address} -> ~{UC_write_to_pc}
- J11 pad 9: unconnected-(J11-Pin_9-Pad9) -> ~{UC_read_mem_const}
- J12 pad 13: ~{UC_write_address} -> ~{UC_write_to_pc}
- J12 pad 9: unconnected-(J12-Pin_9-Pad9) -> ~{UC_read_mem_const}
- J13 pad 13: ~{UC_write_address} -> ~{UC_write_to_pc}
- J13 pad 9: unconnected-(J13-Pin_9-Pad9) -> ~{UC_read_mem_const}
- J14 pad 13: ~{UC_write_address} -> ~{UC_write_to_pc}
- J14 pad 9: unconnected-(J14-Pin_9-Pad9) -> ~{UC_read_mem_const}
- J15 pad 13: ~{UC_write_address} -> ~{UC_write_to_pc}
- J15 pad 9: unconnected-(J15-Pin_9-Pad9) -> ~{UC_read_mem_const}
- J16 pad 13: ~{UC_write_address} -> ~{UC_write_to_pc}
- J16 pad 9: unconnected-(J16-Pin_9-Pad9) -> ~{UC_read_mem_const}
- J17 pad 13: ~{UC_write_address} -> ~{UC_write_to_pc}
- J17 pad 9: unconnected-(J17-Pin_9-Pad9) -> ~{UC_read_mem_const}
- J18 pad 13: ~{UC_write_address} -> ~{UC_write_to_pc}
- J18 pad 9: unconnected-(J18-Pin_9-Pad9) -> ~{UC_read_mem_const}
- J7 pad 13: ~{UC_write_address} -> ~{UC_write_to_pc}
- J7 pad 9: unconnected-(J7-Pin_9-Pad9) -> ~{UC_read_mem_const}
- R30 pad 1: ~{UC_write_address} -> ~{UC_write_to_pc}
- U12 pad 2: INS_{0} -> Net-(U12-D0)
- U16 pad 10: +5V -> INS_{0}
- U16 pad 11: ULA_ENABLE -> unconnected-(U16-Pad11)
- U16 pad 13: ~{UC_ula_enable} -> +5V
- U16 pad 4: +5V -> high_cycle
- U16 pad 5: +5V -> INS_{0}
- U16 pad 6: unconnected-(U16-Pad6) -> Net-(U12-D0)
- U16 pad 8: unconnected-(U16-Pad8) -> Net-(U18-I0a)
- U16 pad 9: +5V -> high_cycle
- U18 pad 1: ~{UC_write_address} -> write_address
- U18 pad 19: ~{UC_write_address} -> write_address
- U18 pad 2: INS_{0} -> Net-(U18-I0a)
- U19 pad 5: Net-(D26-K) -> ~{UC_read_mem_const}
- U19 pad 6: UC_const_boot_addr -> UC_read_mem_const
- U25 pad 11: unconnected-(U25-Pad11) -> WR_ADDR_0
- U25 pad 12: +5V -> Net-(U25-Pad12)
- U25 pad 13: +5V -> ~{UC_write_to_pc}
- U25 pad 2: Net-(U25-Pad2) -> Net-(U25-Pad12)
- U25 pad 5: UC_const_boot_addr -> select_opcode_reset
- U27 pad 9: ~{CLOCK} -> CLOCK
- U30 pad 6: CLOCK -> +5V
- U4 pad 1: Net-(D26-K) -> ULA_ENABLE
- U4 pad 2: reset_low_cycle -> ~{condition_true}
- U4 pad 3: reset_high_cycle -> ~{UC_ula_enable}
- U4 pad 4: Net-(U25-Pad2) -> Net-(U25-Pad12)
Routing:
- net +5V: track 848.9 -> 0.00 mm
- net low_cycle: track 410.6 -> 0.00 mm, vias 6 -> 0
- net high_cycle: track 335.9 -> 0.00 mm, vias 5 -> 0
- net fetch_clock: track 330.9 -> 0.00 mm, vias 3 -> 0
- net ~{UC_restart_cycle}: track 301.2 -> 0.00 mm, vias 2 -> 0
- net select_opcode_int: track 284.5 -> 0.00 mm, vias 1 -> 0
- net ~{UC_pcia_swap}: track 278.1 -> 0.00 mm, vias 3 -> 0
- net ~{UC_extended_opcode}: track 245.1 -> 0.00 mm, vias 2 -> 0
- net ~{UC_write_address}: track 209.2 -> 0.00 mm, vias 2 -> 0
- net ~{UC_read_addr_src_reg}: track 208.9 -> 0.00 mm, vias 2 -> 0
- net ~{UC_write_enable}: track 203.2 -> 0.00 mm, vias 2 -> 0
- net ~{UC_int_ready}: track 189.5 -> 0.00 mm, vias 2 -> 0
- net fetch_cycle: track 177.6 -> 0.00 mm, vias 3 -> 0
- net ~{UC_ula_enable}: track 176.7 -> 0.00 mm, vias 1 -> 0
- net Net-(U29A-C): track 169.0 -> 0.00 mm, vias 2 -> 0
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Other:
- board text added: "MEM[CONST]"
- board text added: "MEM[PC]"
- board text added: "PC"

Commit message: mais simulações e ajustes no pcb; falta o sinal de WRITE durante o reset e interrupt
Parts:
- removed C3: 100nF, Capacitor_THT:C_Disc_D5.1mm_W3.2mm_P5.00mm
- removed D10, D11, D12, D16, D17, D18, D19, D20, D21, D22, D23, D5, D6, D7, D9: 1N4148, Diode_THT:D_DO-35_SOD27_P7.62mm_Horizontal
- removed R13, R14, R5, R6, R7, R8: 1K, Resistor_THT:R_Axial_DIN0207_L6.3mm_D2.5mm_P7.62mm_Horizontal
- removed R2, R23, R24, R25, R26, R27, R28, R29, R30, R31, R32, R33, R35: 10K, Resistor_THT:R_Axial_DIN0207_L6.3mm_D2.5mm_P7.62mm_Horizontal
- removed U3: 74HC04, Package_DIP:DIP-14_W7.62mm
- added C13: 100nF, Capacitor_THT:C_Disc_D5.1mm_W3.2mm_P5.00mm, F.Cu at (52.0, 165.6)
- added C15: 100nF, Capacitor_THT:C_Disc_D5.1mm_W3.2mm_P5.00mm, F.Cu at (68.6, 165.6)
- added C17: 100nF, Capacitor_THT:C_Disc_D5.1mm_W3.2mm_P5.00mm, F.Cu at (85.2, 173.4)
- added D3: WRITE, LED_THT:LED_D5.0mm, F.Cu at (139.1, 222.2)
- added RN1: 10K, Resistor_THT:R_Array_SIP9, F.Cu at (26.7, 177.2)
- added RN2: 10K, Resistor_THT:R_Array_SIP5, F.Cu at (26.7, 182.2)
- added RN3: 10K, Resistor_THT:R_Array_SIP5, F.Cu at (160.0, 73.0)
- added RN4: 10K, Resistor_THT:R_Array_SIP5, F.Cu at (160.0, 58.4)
- added RN5: 10K, Resistor_THT:R_Array_SIP5, F.Cu at (160.0, 43.8)
- added RN6: 10K, Resistor_THT:R_Array_SIP6, F.Cu at (158.8, 122.6)
- added RN7: 10K, Resistor_THT:R_Array_SIP6, F.Cu at (158.8, 118.1)
- added RN8: 1K, Resistor_THT:R_Array_SIP9, F.Cu at (108.0, 215.3)
- added U13: 74LS244, Package_DIP:DIP-20_W7.62mm, F.Cu at (49.5, 169.5)
- added U15: 74LS244, Package_DIP:DIP-20_W7.62mm, F.Cu at (66.0, 169.5)
- added U17: 74LS125, Package_DIP:DIP-14_W7.62mm, F.Cu at (82.5, 177.2)
- D1: value PWR -> POWER
- D4: value 1N4148 -> ULA; footprint Diode_THT:D_DO-35_SOD27_P7.62mm_Horizontal -> LED_THT:LED_D5.0mm
- moved D4 120.5 mm to (146.1, 222.2), turned to 0 degrees
- moved SW1 35.1 mm to (31.1, 157.5), turned to 0 degrees
- moved SW3 32.9 mm to (31.1, 170.8), turned to 0 degrees
- moved D24 32.4 mm to (97.2, 222.2)
- moved R34 21.7 mm to (104.1, 215.3), turned to 180 degrees
- moved D27 17.8 mm to (132.1, 222.2)
- moved D25 14.6 mm to (125.1, 222.2)
- moved SW6 13.6 mm to (31.1, 184.2), turned to 0 degrees
- moved D1 8.25 mm to (153.0, 222.2)
- moved D2 6.35 mm to (104.1, 222.2)
- moved D13 3.17 mm to (111.1, 222.2)
Connections:
- D1 pad 1: GND -> Net-(D1-K)
- D1 pad 2: Net-(D1-A) -> +5V
- D13 pad 1: GND -> Net-(D13-K)
- D13 pad 2: Net-(D13-A) -> low_cycle
- D14 pad 1: GND -> Net-(D14-K)
- D14 pad 2: Net-(D14-A) -> high_cycle
- D2 pad 1: GND -> Net-(D2-K)
- D2 pad 2: Net-(D2-A) -> fetch_cycle
- D25 pad 1: GND -> Net-(D25-K)
- D25 pad 2: Net-(D25-A) -> INT_REQUEST
- D27 pad 1: GND -> Net-(D27-K)
- D27 pad 2: Net-(D27-A) -> int_pending
- D4 pad 1: RD_ADDR_1 -> Net-(D4-K)
- D4 pad 2: Net-(D4-A) -> ULA_ENABLE
- J4 pad 16: unconnected-(J4-Pin_16-Pad16) -> reset_sync
- SW1 pad 1: UC_read_mem_const -> +5V
- SW1 pad 2: UC_read_mem_const -> +5V
- SW1 pad 3: UC_read_mem_const -> +5V
- SW1 pad 4: UC_read_mem_const -> +5V
- SW1 pad 5: Net-(D4-A) -> Net-(RN1-R5)
- SW3 pad 1: fetch_cycle -> +5V
- SW3 pad 2: fetch_cycle -> +5V
- SW3 pad 3: fetch_cycle -> +5V
- SW3 pad 4: fetch_cycle -> +5V
- SW6 pad 1: write_to_pc -> +5V
- SW6 pad 2: write_to_pc -> +5V
- SW6 pad 3: write_to_pc -> +5V
- SW6 pad 4: write_to_pc -> +5V
- U1 pad 11: ~{UC_restart_cycle} -> Net-(U1-~{LOAD})
- U12 pad 1: ~{UC_read_addr_src_reg} -> GND
- U12 pad 15: RD_ADDR_4 -> Net-(U12-Q4)
- U12 pad 16: RD_ADDR_3 -> Net-(U12-Q3)
- U12 pad 17: RD_ADDR_2 -> Net-(U12-Q2)
- U12 pad 18: RD_ADDR_1 -> Net-(U12-Q1)
- U12 pad 19: RD_ADDR_0 -> Net-(U12-Q0)
- U12 pad 2: Net-(U12-D0) -> INS_{0}
- U16 pad 5: INS_{0} -> Net-(U12-Q0)
- U16 pad 6: Net-(U12-D0) -> Net-(U15-I0a)
- U19 pad 1: ~{UC_save_cond_reg} -> +5V
- U19 pad 12: Net-(D23-K) -> ~{restart_cycle}
- U19 pad 2: Net-(U19-Pad2) -> unconnected-(U19-Pad2)
- U19 pad 3: ~{UC_clear_cond_reg} -> ~{UC_save_cond_reg}
- U19 pad 4: Net-(U19-Pad4) -> Net-(U28A-C)
- U19 pad 5: ~{UC_read_mem_const} -> fetch_cycle
- U19 pad 6: UC_read_mem_const -> ~{fetch_cycle}
- U2 pad 15: unconnected-(U2-Y0-Pad15) -> reset_sync
- U20 pad 4: Net-(U19-Pad2) -> ~{UC_write_enable}
- U20 pad 5: ~{CLOCK} -> ~{UC_ula_enable}
- U20 pad 6: Net-(U28A-C) -> write_address
- U27 pad 11: unconnected-(U27-Pad11) -> Net-(U1-~{LOAD})
- U27 pad 12: +5V -> ~{UC_restart_cycle}
- U27 pad 13: +5V -> ~{restart_cycle}
- U28 pad 1: Net-(U28A-~{R}) -> ~{UC_clear_cond_reg}
- U29 pad 1: ~{UC_clear_pending_int} -> ~{UC_int_ready}
- U30 pad 14: ~{UC_clear_pending_int} -> unconnected-(U30-O1-Pad14)
- U32 pad 6: Net-(D20-K) -> Net-(U32-E3)
- U4 pad 11: Net-(U19-Pad4) -> +5V
- U4 pad 12: RESET -> +5V
- U4 pad 13: Net-(U28A-~{R}) -> unconnected-(U4-Pad13)
- U5 pad 1: ~{UC_write_enable} -> +5V
- U5 pad 10: +5V -> high_cycle
- U5 pad 2: ~{UC_ula_enable} -> +5V
- U5 pad 3: write_address -> unconnected-(U5-Pad3)
- U5 pad 4: +5V -> low_cycle
- U5 pad 5: +5V -> fetch_cycle
- U5 pad 6: unconnected-(U5-Pad6) -> Net-(U5-Pad6)
- U5 pad 8: unconnected-(U5-Pad8) -> Net-(U32-E3)
- U5 pad 9: +5V -> Net-(U5-Pad6)
