File: pcb_v2/sysbusa/sysbusa.kicad_pcb (KiCad board)
At the start: 2 copper layers, 96 parts, among them J1 bus ula 2, J10 bus rf16 3, J11 bus clu 2, J12 bus clu 3, J19 9V 1A, J2 bus ula 1, J20 VOLTMETER, J21 AMPMETER, J22 bus ioc 2, J23 bus ioc 1, J24 bus ioc 3, J26 bus clock, J3 bus rf16 1, J4 bus rf16 2, J5 bus mem 1, J6 bus mem 2, J7 bus clu 1, J8 bus mgrf 1, J9 bus mgrf 2, Q1 BC548, Q2 BC548, SW1 RESET, U1 MC14495P, U10 MC14495P, U11 ADDR N1, U12 DATA N0, U13 MC14495P, U14 RDADDR_LOW, U17 RDADDR_HIGH, U2 ADDR N3, U21 MC14495P, U22 WRADDR_HIGH, U23 WRADDR_LOW, U3 MC14495P, U31 MC14495P, U34 LM7805, U4 ADDR N2, U5 74LS08, U6 MC14495P, U7 DATA N1, U8 MC14495P, U9 ADDR N0

Commit message: padronização de conector de IO; ideias para o layout do backplane
Parts:
- removed R1, R2, R3, R4, R5: 10K, Resistor_THT:R_Axial_DIN0207_L6.3mm_D2.5mm_P7.62mm_Horizontal
- moved R14 172.5 mm to (45.7, 114.3), turned to 90 degrees
- moved R13 170.3 mm to (47.6, 103.5), turned to 90 degrees
- moved R11 169.9 mm to (49.5, 114.3), turned to 90 degrees
- moved J20 168.0 mm to (123.7, 125.1)
- moved J21 168.0 mm to (130.8, 125.1)
- moved J19 168.0 mm to (116.5, 125.1)
- moved R10 157.5 mm to (51.4, 103.5), turned to 90 degrees
- moved R9 154.0 mm to (53.3, 114.3), turned to 90 degrees
- moved R8 152.7 mm to (55.2, 103.5), turned to 90 degrees
- moved R7 149.9 mm to (57.1, 114.3), turned to 90 degrees
- moved R51 148.8 mm to (92.1, 106.7), turned to -90 degrees
- moved R6 148.3 mm to (59.1, 103.5), turned to 90 degrees
- moved R50 148.1 mm to (94.0, 95.9), turned to -90 degrees
- moved U5 144.9 mm to (134.6, 81.3)
- moved R49 144.1 mm to (95.9, 106.7), turned to -90 degrees
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- renumbered C6 to C2, C2 to C3, C3 to C5, C4 to C6, C5 to C8
Connections:
- J11 pad 15: CLOCK -> unconnected-(J11-Pin_15-Pad15)
- J12 pad 13: unconnected-(J12-Pin_13-Pad13) -> ~{CLOCK}
- J12 pad 15: unconnected-(J12-Pin_15-Pad15) -> CLOCK
- J24 pad 1: WR_ADDR_0 -> unconnected-(J24-Pin_1-Pad1)
- J24 pad 11: unconnected-(J24-Pin_11-Pad11) -> WR_ADDR_3
- J24 pad 13: unconnected-(J24-Pin_13-Pad13) -> WR_ADDR_4
- J24 pad 3: WR_ADDR_1 -> unconnected-(J24-Pin_3-Pad3)
- J24 pad 5: WR_ADDR_2 -> WR_ADDR_0
- J24 pad 7: WR_ADDR_3 -> WR_ADDR_1
- J24 pad 9: WR_ADDR_4 -> WR_ADDR_2
- J26 pad 14: unconnected-(J26-Pin_14-Pad14) -> ~{CLOCK}
- U5 pad 12: unconnected-(U5-Pad12) -> +5V
- U5 pad 13: unconnected-(U5-Pad13) -> +5V
- U5 pad 4: unconnected-(U5-Pad4) -> +5V
- U5 pad 5: unconnected-(U5-Pad5) -> +5V
Other:
- board outline added: 198.1 x 114.3 mm

Commit message: definindo o layout para empilhar as placas
Parts:
- added R1: 470R, Resistor_THT:R_Axial_DIN0207_L6.3mm_D2.5mm_P7.62mm_Horizontal, F.Cu at (123.8, 116.2)
- SW1: footprint Button_Switch_THT:SW_PUSH_6mm -> Connector_Molex:Molex_KK-254_AE-6410-02A_1x02_P2.54mm_Vertical
- moved SW1 185.7 mm to (36.2, 61.0)
- moved D32 181.9 mm to (36.2, 124.5)
- moved J2 178.8 mm to (216.5, 110.5), turned to 180 degrees
- moved C14 177.9 mm to (35.6, 102.2)
- moved C11 177.1 mm to (35.6, 91.4)
- moved U34 177.1 mm to (36.2, 113.0)
- moved J23 174.1 mm to (216.5, 50.8), turned to 180 degrees
- moved J3 173.4 mm to (216.5, 80.6), turned to 180 degrees
- moved U12 167.8 mm to (62.2, 137.8)
- moved C2 153.5 mm to (60.4, 88.3)
- moved U7 147.8 mm to (51.4, 137.8)
- moved U8 144.2 mm to (58.4, 104.8)
- moved C8 144.2 mm to (61.0, 101.0)
- moved J1 142.8 mm to (208.9, 110.5), turned to 180 degrees
- moved J24 136.9 mm to (208.9, 50.8), turned to 180 degrees
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Connections:
- Q1 pad 1: GND -> Net-(Q1-C)
Other:
- board size 198.1 x 114.3 mm -> 198.1 x 128.3 mm
- board text added: "ADDRESS BUS"
- board text added: "CLOCK"
- board text added: "CLU"
- board text added: "DATA BUS"
- board text added: "IOC"
- board text added: "MEM"
- board text added: "MGRF"
- board text added: "READ"
- board text added: "RF16"
- board text added: "ULA"
- board text added: "WRITE"

Commit message: refazendo os pcbs para caber em folha A4
Parts:
- removed J8: bus mgrf 1, Connector_PinHeader_2.54mm:PinHeader_2x08_P2.54mm_Vertical
- removed J9: bus mgrf 2, Connector_PinHeader_2.54mm:PinHeader_2x08_P2.54mm_Vertical
- added R2: 10K, Resistor_THT:R_Axial_DIN0207_L6.3mm_D2.5mm_P7.62mm_Horizontal, F.Cu at (238.1, 72.4)
- added R25: 10K, Resistor_THT:R_Axial_DIN0207_L6.3mm_D2.5mm_P7.62mm_Horizontal, F.Cu at (245.7, 72.4)
- added R3: 10K, Resistor_THT:R_Axial_DIN0207_L6.3mm_D2.5mm_P7.62mm_Horizontal, F.Cu at (240.0, 62.2)
- added R4: 10K, Resistor_THT:R_Axial_DIN0207_L6.3mm_D2.5mm_P7.62mm_Horizontal, F.Cu at (241.9, 72.4)
- added R5: 10K, Resistor_THT:R_Axial_DIN0207_L6.3mm_D2.5mm_P7.62mm_Horizontal, F.Cu at (243.8, 62.2)
- J1: value bus ula 2 -> ula_2
- J2: value bus ula 1 -> ula_1
- U11, U12, U14, U17, U2, U22, U23, U4, U7, U9: footprint 7segdisplay:1-digit-13mm -> Display_7Segment:Sx39-1xxxxx
- moved C11 252.1 mm to (287.7, 85.7), turned to 90 degrees
- moved J20 241.3 mm to (277.5, 85.1), turned to 180 degrees
- moved J21 232.7 mm to (268.6, 85.1), turned to 180 degrees
- moved SW1 222.3 mm to (257.2, 85.1), turned to 0 degrees
- moved C14 212.8 mm to (247.7, 84.5), turned to -90 degrees
- moved U34 202.6 mm to (236.9, 85.1), turned to 180 degrees
- moved D32 193.3 mm to (225.4, 85.1), turned to 180 degrees
- moved J19 180.3 mm to (207.0, 85.1), turned to 0 degrees
- moved R40 113.5 mm to (283.8, 54.6)
- moved R42 113.5 mm to (280.0, 54.6)
- moved R15 113.5 mm to (250.2, 62.2)
- moved R16 113.5 mm to (252.1, 72.4)
- moved R17 113.5 mm to (254.0, 62.2)
- moved R18 113.5 mm to (255.9, 72.4)
- moved R19 113.5 mm to (257.8, 62.2)
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Connections:
- R1 pad 1: Net-(Q1-C) -> Net-(Q1-E)
- R20 pad 1: Net-(Q2-C) -> Net-(Q2-E)
- U22 pad 3: Net-(Q2-E) -> Net-(Q2-C)
- U22 pad 8: Net-(Q2-E) -> Net-(Q2-C)
- U23 pad 3: Net-(Q1-E) -> Net-(Q1-C)
- U23 pad 8: Net-(Q1-E) -> Net-(Q1-C)
Other:
- board size 198.1 x 128.3 mm -> 297 x 75 mm
- board text removed: "MGRF"

Commit message: posicionamento dos conectores com os demais módulos
Parts:
- J1: value ula_2 -> bus ula 2
- J19: value 9V 1A -> 9V 2A; footprint Connector_Molex:Molex_KK-254_AE-6410-02A_1x02_P2.54mm_Vertical -> Connector_JST:JST_XH_B2B-XH-A_1x02_P2.50mm_Vertical
- J2: value ula_1 -> bus ula 1
- J20, J21, SW1: footprint Connector_Molex:Molex_KK-254_AE-6410-02A_1x02_P2.54mm_Vertical -> Connector_JST:JST_XH_B2B-XH-A_1x02_P2.50mm_Vertical
- moved R20 102.7 mm to (198.1, 73.7)
- moved R22 102.7 mm to (194.3, 73.7)
- moved R1 102.7 mm to (186.7, 73.7)
- moved R21 102.7 mm to (190.5, 73.7)
- moved C5 76.8 mm to (227.3, 69.3), turned to -90 degrees
- moved U5 75.4 mm to (222.9, 66.7), turned to -90 degrees
- moved Q1 72.6 mm to (179.7, 67.9)
- moved Q2 72.6 mm to (173.4, 67.9)
- moved J19 72.2 mm to (278.8, 92.7), turned to 180 degrees
- moved C11 51.6 mm to (236.9, 94.6)
- moved C2 42.1 mm to (202.6, 92.1)
- moved R24 40.6 mm to (202.6, 84.5), turned to 0 degrees
- moved D32 35.1 mm to (259.7, 92.7), turned to 0 degrees
- moved SW1 31.4 mm to (287.7, 92.7), turned to 180 degrees
- moved U11 29.7 mm to (86.2, 85.0)
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Other:
- outline, holes or cut-outs redrawn

Commit message: reposicionado o conector para a ULA
Parts:
- moved J5 116.2 mm to (108.6, 34.3)
- moved J6 116.2 mm to (108.6, 45.1)
- moved J1 38.1 mm to (200.7, 44.5)
- moved J11 38.1 mm to (156.2, 54.6)
- moved J12 38.1 mm to (156.2, 43.8)
- moved J7 38.1 mm to (156.2, 33.0)
- moved J2 38.0 mm to (200.6, 33.0)
Other:
- outline, holes or cut-outs redrawn
Changed lines of the file:
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@@
 	(footprint "Connector_PinHeader_2.54mm:PinHeader_2x08_P2.54mm_Vertical"
 		(layer "F.Cu")
-		(at 162.56 45.72 90)
+		(at 200.66 44.45 90)
 		(descr "Through hole straight pin header, 2x08, 2.54mm pitch, double rows")
 		(tags "Through hole pin header THT 2x08 2.54mm double row")
@@
 	(footprint "Connector_PinHeader_2.54mm:PinHeader_2x08_P2.54mm_Vertical"
 		(layer "F.Cu")
-		(at 118.11 44.45 90)
+		(at 156.21 43.815 90)
 		(descr "Through hole straight pin header, 2x08, 2.54mm pitch, double rows")
 		(tags "Through hole pin header THT 2x08 2.54mm double row")
@@
 	(footprint "Connector_PinHeader_2.54mm:PinHeader_2x08_P2.54mm_Vertical"
 		(layer "F.Cu")
-		(at 162.56 34.29 90)
+		(at 200.58 33.02 90)
 		(descr "Through hole straight pin header, 2x08, 2.54mm pitch, double rows")
 		(tags "Through hole pin header THT 2x08 2.54mm double row")
@@
 	(footprint "Connector_PinHeader_2.54mm:PinHeader_2x08_P2.54mm_Vertical"
 		(layer "F.Cu")
-		(at 118.11 33.655 90)
+		(at 156.21 33.02 90)
 		(descr "Through hole straight pin header, 2x08, 2.54mm pitch, double rows")
 		(tags "Through hole pin header THT 2x08 2.54mm double row")
@@
 	(footprint "Connector_PinHeader_2.54mm:PinHeader_2x08_P2.54mm_Vertical"
 		(layer "F.Cu")
-		(at 224.79 33.02 90)
+		(at 108.585 34.29 90)
 		(descr "Through hole straight pin header, 2x08, 2.54mm pitch, double rows")
 		(tags "Through hole pin header THT 2x08 2.54mm double row")
@@
 	(footprint "Connector_PinHeader_2.54mm:PinHeader_2x08_P2.54mm_Vertical"
 		(layer "F.Cu")
-		(at 118.11 55.245 90)
+		(at 156.21 54.61 90)
 		(descr "Through hole straight pin header, 2x08, 2.54mm pitch, double rows")
 		(tags "Through hole pin header THT 2x08 2.54mm double row")
@@
 	(footprint "Connector_PinHeader_2.54mm:PinHeader_2x08_P2.54mm_Vertical"
 		(layer "F.Cu")
-		(at 224.79 43.815 90)
+		(at 108.585 45.085 90)
 		(descr "Through hole straight pin header, 2x08, 2.54mm pitch, double rows")
 		(tags "Through hole pin header THT 2x08 2.54mm double row")
@@
 	)
 	(gr_rect
-		(start 112.395 27.94)
-		(end 141.605 58.475)
+		(start 102.87 28.575)
+		(end 132.08 48.26)
 		(stroke
 			(width 0.3)
@@
 	)
 	(gr_rect
-		(start 156.845 28.575)
-		(end 186.055 48.895)
+		(start 150.495 27.305)
+		(end 179.705 57.84)
 		(stroke
 			(width 0.3)
@@
 	)
 	(gr_rect
-		(start 219.075 27.305)
-		(end 248.285 46.99)
+		(start 194.945 27.075)
+		(end 224.155 47.395)
 		(stroke
 			(width 0.3)
@@
 		(layer "Edge.Cuts")
 	)
-	(gr_rect
-		(start 280.64 28.75)
-		(end 308.64 34.75)
-		(stroke
-			(width 0.1)
-			(type solid)
-		)
-		(fill no)
-		(layer "Edge.Cuts")
-	)
 	(gr_circle
 		(center 312.59 31.4)
@@
 		)
 	)
-	(gr_text "WRITE"
-		(at 124.9675 81.1525 0)
+	(gr_text "MEM"
+		(at 116.205 50.8 0)
 		(layer "F.SilkS")
 		(effects
@@
 		)
 	)
-	(gr_text "CLU"
-		(at 127 60.325 0)
+	(gr_text "WRITE"
+		(at 124.9675 81.1525 0)
 		(layer "F.SilkS")
 		(effects
@@
 		)
 	)
-	(gr_text "ULA"
-		(at 171.45 50.8 0)
+	(gr_text "CLU"
+		(at 165.1 59.69 0)
 		(layer "F.SilkS")
 		(effects
@@
 		)
 	)
-	(gr_text "MEM"
-		(at 233.68 48.895 0)
+	(gr_text "ULA"
+		(at 209.55 50.165 0)
 		(layer "F.SilkS")
 		(effects

Commit message: inicio do layout da pcb
Parts:
- removed C5: 100nF, Capacitor_THT:C_Disc_D5.1mm_W3.2mm_P5.00mm
- removed R10, R11, R13, R14, R15, R16, R17, R18, R19, R2, R25, R3, R36, R37, R38, R39, R4, R40, R41, R42, R43, R44, R45, R46, R47, R48, R49, R5, R50, R51, R6, R7, R8, R9: 10K, Resistor_THT:R_Axial_DIN0207_L6.3mm_D2.5mm_P7.62mm_Horizontal
- removed U5: 74LS08, Package_DIP:DIP-14_W7.62mm
- added RN1: 10K, Resistor_THT:R_Array_SIP9, F.Cu at (247.0, 31.8)
- added RN2: 10K, Resistor_THT:R_Array_SIP9, F.Cu at (247.0, 42.5)
- added RN3: 10K, Resistor_THT:R_Array_SIP9, F.Cu at (247.0, 58.4)
- J19: value 9V 2A -> 9V 1A
- moved J24 25.6 mm to (255.3, 59.7), turned to 90 degrees
- moved J4 25.6 mm to (285.8, 59.7), turned to 90 degrees
- moved R12 23.6 mm to (143.5, 62.2), turned to 180 degrees
- moved Q1 21.7 mm to (177.2, 89.5)
- moved Q2 21.7 mm to (170.8, 89.5)
- moved R1 21.7 mm to (184.2, 95.2)
- moved R20 21.7 mm to (195.6, 95.2)
- moved R21 21.7 mm to (188.0, 95.2)
- moved R22 21.7 mm to (191.8, 95.2)
- moved J22 19.6 mm to (255.3, 43.8), turned to 90 degrees
- moved J10 19.6 mm to (285.8, 43.8), turned to 90 degrees
- moved J23 18.0 mm to (255.3, 33.0), turned to 90 degrees
- moved J3 18.0 mm to (285.8, 33.0), turned to 90 degrees
- moved U1 5.12 mm to (52.1, 52.7)
- moved J11 5.08 mm to (156.2, 59.7)
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Connections:
- C2 pad 2: Net-(C2-Pad2) -> RESET
- R24 pad 1: Net-(C2-Pad2) -> RESET
- SW1 pad 2: Net-(C2-Pad2) -> RESET
Routing:
- net +5V: track 0.00 -> 526.1 mm
- net CLOCK: track 0.00 -> 355.2 mm, vias 0 -> 6
- net DATA_{7}: track 0.00 -> 335.8 mm, vias 0 -> 7
- net DATA_{6}: track 0.00 -> 319.8 mm, vias 0 -> 7
- net DATA_{5}: track 0.00 -> 315.6 mm, vias 0 -> 7
- net DATA_{4}: track 0.00 -> 313.0 mm, vias 0 -> 7
- net DATA_{0}: track 0.00 -> 310.6 mm, vias 0 -> 6
- net DATA_{2}: track 0.00 -> 305.0 mm, vias 0 -> 7
- net DATA_{3}: track 0.00 -> 302.1 mm, vias 0 -> 7
- net DATA_{1}: track 0.00 -> 300.3 mm, vias 0 -> 6
- net ADDR_{14}: track 0.00 -> 292.1 mm, vias 0 -> 3
- net ADDR_{12}: track 0.00 -> 287.4 mm, vias 0 -> 4
- net ADDR_{10}: track 0.00 -> 281.4 mm, vias 0 -> 4
- net ADDR_{13}: track 0.00 -> 280.3 mm, vias 0 -> 4
- net ADDR_{15}: track 0.00 -> 279.9 mm, vias 0 -> 2
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- added copper zone on B.Cu, net GND
- added copper zone on F.Cu, net GND

Commit message: concluída a primeira versão do layout do pcb; rever o circuito de reset
Parts:
- moved R12 49.5 mm to (180.3, 95.2), turned to 90 degrees
- moved Q1 7.75 mm to (170.8, 85.1)
- moved R1 7.62 mm to (184.2, 87.6), turned to -90 degrees
- moved R23 6.98 mm to (220.3, 83.8), turned to 180 degrees
- moved Q2 2.54 mm to (170.8, 92.1)
- moved C2 2.50 mm to (204.5, 91.4), turned to 180 degrees
- moved C11 1.95 mm to (236.9, 92.1), turned to 180 degrees
- moved C14 0.95 mm to (226.8, 92.1), turned to 0 degrees
- moved U34 0.63 mm to (246.4, 92.1)
Routing:
- net +5V: track 526.1 -> 743.6 mm
- net RESET: track 143.1 -> 338.1 mm, vias 2 -> 3
- net WR_ADDR_1: track 163.2 -> 274.2 mm, vias 3 -> 6
- net WR_ADDR_0: track 166.8 -> 272.1 mm, vias 3 -> 6
- net WR_ADDR_4: track 150.6 -> 254.2 mm, vias 3 -> 6
- net WR_ADDR_2: track 159.6 -> 262.3 mm, vias 3 -> 5
- net WR_ADDR_3: track 155.8 -> 255.7 mm, vias 3 -> 5
- net RD_ADDR_4: track 158.0 -> 233.0 mm, vias 2 -> 5
- net Net-(J21-Pin_1): track 0.00 -> 73.4 mm
- net Net-(Q2-C): track 0.00 -> 61.0 mm
- net Net-(Q1-C): track 0.00 -> 56.0 mm
- net Net-(R12-Pad1): track 0.00 -> 48.2 mm, vias 0 -> 1
- net RD_ADDR_3: track 197.1 -> 233.6 mm, vias 3 -> 5
- net RD_ADDR_2: track 205.0 -> 240.0 mm, vias 3 -> 5
- net RD_ADDR_1: track 199.0 -> 233.6 mm, vias 3 -> 5
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
Commit message: revisão na posição dos conectores
Parts:
- moved R23 17.6 mm to (203.2, 87.6), turned to -90 degrees
- moved C2 15.9 mm to (220.3, 90.8), turned to -90 degrees
- moved R24 4.58 mm to (199.4, 87.6), turned to -90 degrees
- moved D1 0.90 mm to (210.8, 92.1), turned to 180 degrees
Routing:
- net RESET: track 338.1 -> 343.7 mm
- net +5V: track 743.6 -> 739.2 mm
- net Net-(D1-A): track 8.15 -> 6.40 mm
Other:
- board text added: "A"
- board text added: "B"
- board text added: "C"
- board text added: "Rev.A1 maio/2026"
- board text added: "SYSBUS"
- board text added: "ULA8"
- board text removed: "ULA"
