File: pcb_v2/sysbusa/sysbusa.kicad_sch (KiCad schematic)
At the start: 67 parts, among them J1 bus ula 2, J10 bus rf16 3, J11 bus clu 2, J12 bus clu 3, J19 9V 1A, J2 bus ula 1, J20 VOLTS, J21 AMPS, J22 bus ioc 2, J23 bus ioc 1, J24 bus ioc 3, J26 bus clock, J3 bus rf16 1, J4 bus rf16 2, J5 bus mem 1, J6 bus mem 2, J7 bus clu 1, Q1 BC548, Q2 BC548, SW1 RESET, U1 MC14495P, U10 MC14495P, U11 ADDR N1, U12 DATA N0, U13 MC14495P, U14 RDADDR_LOW, U17 RDADDR_HIGH, U2 ADDR N3, U21 MC14495P, U22 WRADDR_HIGH, U23 WRADDR_LOW, U3 MC14495P, U31 MC14495P, U34 LM7805, U4 ADDR N2, U5 NE555P, U6 MC14495P, U7 DATA N1, U8 MC14495P, U9 ADDR N0

Commit message: usando um componente com as dimensões do conector de cabo flat, para impedir erros de posicionamento
Parts:
- J1, J10, J11, J12, J2, J22, J23, J24, J26, J3, J4, J5, J6, J7: footprint Connector_PinHeader_2.54mm:PinHeader_2x08_P2.54mm_Vertical -> edge_connector:conector 02x08
Changed lines of the file:
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@@
 			)
 		)
-		(property "Footprint" "Connector_PinHeader_2.54mm:PinHeader_2x08_P2.54mm_Vertical"
+		(property "Footprint" "edge_connector:conector 02x08"
 			(at 34.29 29.21 0)
 			(effects
@@
 			)
 		)
-		(property "Footprint" "Connector_PinHeader_2.54mm:PinHeader_2x08_P2.54mm_Vertical"
+		(property "Footprint" "edge_connector:conector 02x08"
 			(at 189.23 60.96 0)
 			(effects
@@
 			)
 		)
-		(property "Footprint" "Connector_PinHeader_2.54mm:PinHeader_2x08_P2.54mm_Vertical"
+		(property "Footprint" "edge_connector:conector 02x08"
 			(at 33.02 153.67 0)
 			(effects
@@
 			)
 		)
-		(property "Footprint" "Connector_PinHeader_2.54mm:PinHeader_2x08_P2.54mm_Vertical"
+		(property "Footprint" "edge_connector:conector 02x08"
 			(at 189.23 88.9 0)
 			(effects
@@
 			)
 		)
-		(property "Footprint" "Connector_PinHeader_2.54mm:PinHeader_2x08_P2.54mm_Vertical"
+		(property "Footprint" "edge_connector:conector 02x08"
 			(at 137.16 59.69 0)
 			(effects
@@
 			)
 		)
-		(property "Footprint" "Connector_PinHeader_2.54mm:PinHeader_2x08_P2.54mm_Vertical"
+		(property "Footprint" "edge_connector:conector 02x08"
 			(at 137.16 29.21 0)
 			(effects
@@
 			)
 		)
-		(property "Footprint" "Connector_PinHeader_2.54mm:PinHeader_2x08_P2.54mm_Vertical"
+		(property "Footprint" "edge_connector:conector 02x08"
 			(at 33.02 60.96 0)
 			(effects
@@
 			)
 		)
-		(property "Footprint" "Connector_PinHeader_2.54mm:PinHeader_2x08_P2.54mm_Vertical"
+		(property "Footprint" "edge_connector:conector 02x08"
 			(at 33.02 124.46 0)
 			(effects
@@
 			)
 		)
-		(property "Footprint" "Connector_PinHeader_2.54mm:PinHeader_2x08_P2.54mm_Vertical"
+		(property "Footprint" "edge_connector:conector 02x08"
 			(at 189.23 29.21 0)
 			(effects
@@
 			)
 		)
-		(property "Footprint" "Connector_PinHeader_2.54mm:PinHeader_2x08_P2.54mm_Vertical"
+		(property "Footprint" "edge_connector:conector 02x08"
 			(at 34.29 92.71 0)
 			(effects
@@
 			)
 		)
-		(property "Footprint" "Connector_PinHeader_2.54mm:PinHeader_2x08_P2.54mm_Vertical"
+		(property "Footprint" "edge_connector:conector 02x08"
 			(at 87.63 60.96 0)
 			(effects
@@
 			)
 		)
-		(property "Footprint" "Connector_PinHeader_2.54mm:PinHeader_2x08_P2.54mm_Vertical"
+		(property "Footprint" "edge_connector:conector 02x08"
 			(at 87.63 29.21 0)
 			(effects
@@
 			)
 		)
-		(property "Footprint" "Connector_PinHeader_2.54mm:PinHeader_2x08_P2.54mm_Vertical"
+		(property "Footprint" "edge_connector:conector 02x08"
 			(at 135.89 96.52 0)
 			(effects
@@
 			)
 		)
-		(property "Footprint" "Connector_PinHeader_2.54mm:PinHeader_2x08_P2.54mm_Vertical"
+		(property "Footprint" "edge_connector:conector 02x08"
 			(at 87.63 88.9 0)
 			(effects
