File: pcb_v3/m16rf/m16rf.kicad_sch (KiCad schematic)
At the start: 55 parts, among them J1 r16_D, J3 r16_A, J4 r16_B, J5 r16_C, J8 bus_rf16_1, J9 bus_rf16_2, U1 74LS125, U10 74LS244, U11 74LS244, U13 74LS02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

Commit message: novo layout para pcb v3
Connections:
- net wr_enable: no longer J3.6 (Pin_6)
- net write renamed write_clock
- net write_clock: now also J3.6 (Pin_6)
Other:
- moved on the sheet: J8, J9
