File: pcb_v3/s16rf/s16rf.kicad_pcb (KiCad board)
At the start: 2 copper layers, 297 x 125 mm, 105 parts, among them J1 r16_D, J2 r16_C, J3 r16_A, J4 r16_B, J5 r16_C, U1 74LS193, U10 74LS193, U11 74LS193, U12 74LS244, U13 74LS193, U14 74LS244, U15 74LS193, U16 74LS244, U17 74LS244, U18 74LS193, U19 74LS193, U2 74LS193, U20 74LS244, U21 74LS193, U22 74LS244, U23 74LS193, U24 74LS244, U25 74LS244, U26 74LS193, U27 74LS193, U28 74LS244, U29 74LS193, U3 74LS193, U30 74LS244, U31 74LS193, U32 74LS244, U33 74LS244, U34 74LS193, U35 74LS193, U36 74LS244, U37 74LS193, U38 74LS244, U39 74LS193, U4 74LS193, U40 74LS244, U41 74LS574, U42 74LS574, U43 74HC238, U44 74LS574, U45 74LS574, U46 74LS138, U47 74LS574, U49 74LS574, U5 74LS244, U50 74LS574, U6 74LS244, U7 74LS244, U8 74LS244, U9 74LS244

Commit message: avançando o layout da placa com os registradores
Parts:
- moved U13 49.2 mm to (97.2, 99.1)
- moved U15 49.2 mm to (110.5, 99.1)
- moved C13 49.2 mm to (99.8, 95.2)
- moved C15 49.2 mm to (113.2, 95.2)
- moved U3 48.2 mm to (40.6, 99.1)
- moved U4 48.2 mm to (54.0, 99.1)
- moved C3 48.2 mm to (43.3, 95.2)
- moved C4 48.2 mm to (56.6, 95.2)
- moved C21 48.1 mm to (163.2, 95.2)
- moved C23 48.1 mm to (176.5, 95.2)
- moved U21 48.1 mm to (160.7, 99.1)
- moved U23 48.1 mm to (174.0, 99.1)
- moved C22 31.2 mm to (189.9, 62.2)
- moved U22 31.2 mm to (187.2, 66.0)
- moved C7 31.0 mm to (69.9, 62.2)
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Connections:
- U12 pad 16: data_{1} -> data_{0}
- U12 pad 18: data_{0} -> data_{1}
- U12 pad 2: sp_count_{0} -> sp_count_{1}
- U12 pad 4: sp_count_{1} -> sp_count_{0}
- U14 pad 16: addr_{9} -> addr_{8}
- U14 pad 18: addr_{8} -> addr_{9}
- U14 pad 2: sp_count_{8} -> sp_count_{9}
- U14 pad 4: sp_count_{9} -> sp_count_{8}
- U16 pad 16: addr_{1} -> addr_{0}
- U16 pad 18: addr_{0} -> addr_{1}
- U16 pad 2: sp_count_{0} -> sp_count_{1}
- U16 pad 4: sp_count_{1} -> sp_count_{0}
- U17 pad 11: zero_count_{12} -> zero_count_{15}
- U17 pad 13: zero_count_{13} -> zero_count_{14}
- U17 pad 15: zero_count_{14} -> zero_count_{12}
- U17 pad 16: data_{1} -> data_{0}
- U17 pad 17: zero_count_{15} -> zero_count_{13}
- U17 pad 18: data_{0} -> data_{1}
- U17 pad 2: zero_count_{8} -> zero_count_{9}
- U17 pad 3: data_{7} -> data_{5}
- U17 pad 4: zero_count_{9} -> zero_count_{8}
- U17 pad 5: data_{6} -> data_{4}
- U17 pad 7: data_{5} -> data_{6}
- U17 pad 9: data_{4} -> data_{7}
- U20 pad 16: data_{1} -> data_{0}
- U20 pad 18: data_{0} -> data_{1}
- U20 pad 2: zero_count_{0} -> zero_count_{1}
- U20 pad 4: zero_count_{1} -> zero_count_{0}
- U22 pad 16: addr_{9} -> addr_{8}
- U22 pad 18: addr_{8} -> addr_{9}
- U22 pad 2: zero_count_{8} -> zero_count_{9}
- U22 pad 4: zero_count_{9} -> zero_count_{8}
- U24 pad 16: addr_{1} -> addr_{0}
- U24 pad 18: addr_{0} -> addr_{1}
- U24 pad 2: zero_count_{0} -> zero_count_{1}
- U24 pad 4: zero_count_{1} -> zero_count_{0}
- U5 pad 11: mar_count_{12} -> mar_count_{15}
- U5 pad 13: mar_count_{13} -> mar_count_{14}
- U5 pad 15: mar_count_{14} -> mar_count_{12}
- U5 pad 16: data_{1} -> data_{0}
- U5 pad 17: mar_count_{15} -> mar_count_{13}
- U5 pad 18: data_{0} -> data_{1}
- U5 pad 2: mar_count_{8} -> mar_count_{9}
- U5 pad 3: data_{7} -> data_{5}
- U5 pad 4: mar_count_{9} -> mar_count_{8}
- U5 pad 5: data_{6} -> data_{4}
- U5 pad 7: data_{5} -> data_{6}
- U5 pad 9: data_{4} -> data_{7}
- U6 pad 16: data_{1} -> data_{0}
- U6 pad 18: data_{0} -> data_{1}
- U6 pad 2: mar_count_{0} -> mar_count_{1}
- U6 pad 4: mar_count_{1} -> mar_count_{0}
- U7 pad 16: addr_{9} -> addr_{8}
- U7 pad 18: addr_{8} -> addr_{9}
- U7 pad 2: mar_count_{8} -> mar_count_{9}
- U7 pad 4: mar_count_{9} -> mar_count_{8}
- U8 pad 16: addr_{1} -> addr_{0}
- U8 pad 18: addr_{0} -> addr_{1}
- U8 pad 2: mar_count_{0} -> mar_count_{1}
- U8 pad 4: mar_count_{1} -> mar_count_{0}
- U9 pad 11: sp_count_{12} -> sp_count_{15}
- U9 pad 13: sp_count_{13} -> sp_count_{14}
- U9 pad 15: sp_count_{14} -> sp_count_{12}
- U9 pad 16: data_{1} -> data_{0}
- U9 pad 17: sp_count_{15} -> sp_count_{13}
- U9 pad 18: data_{0} -> data_{1}
- U9 pad 2: sp_count_{8} -> sp_count_{9}
- U9 pad 3: data_{7} -> data_{5}
- U9 pad 4: sp_count_{9} -> sp_count_{8}
- U9 pad 5: data_{6} -> data_{4}
- U9 pad 7: data_{5} -> data_{6}
- U9 pad 9: data_{4} -> data_{7}
Routing:
- net +5V: track 0.00 -> 637.8 mm
- net addr_{3}: track 154.6 -> 503.7 mm, vias 1 -> 4
- net addr_{4}: track 158.6 -> 501.3 mm, vias 1 -> 4
- net addr_{2}: track 149.3 -> 487.6 mm, vias 1 -> 4
- net addr_{5}: track 153.2 -> 486.2 mm, vias 1 -> 4
- net addr_{0}: track 138.6 -> 471.0 mm, vias 1 -> 4
- net addr_{6}: track 147.9 -> 470.1 mm, vias 1 -> 4
- net addr_{1}: track 143.9 -> 455.6 mm, vias 1 -> 4
- net addr_{7}: track 150.0 -> 454.1 mm, vias 1 -> 4
- net addr_{11}: track 163.6 -> 403.9 mm, vias 1 -> 4
- net addr_{12}: track 174.0 -> 407.0 mm, vias 1 -> 4
- net addr_{10}: track 158.3 -> 387.9 mm, vias 1 -> 4
- net addr_{13}: track 168.1 -> 391.0 mm, vias 1 -> 4
- net addr_{8}: track 150.6 -> 371.8 mm, vias 1 -> 4
- net addr_{14}: track 161.4 -> 375.0 mm, vias 1 -> 4
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
Commit message: finalização da primeira fase de layout do pcb
Parts:
- moved U39 37.0 mm to (288.2, 99.1)
- moved C39 37.0 mm to (290.8, 95.2)
- moved U37 36.9 mm to (275.0, 99.1)
- moved C37 36.9 mm to (277.6, 95.2)
- moved C29 35.5 mm to (221.1, 95.2)
- moved U29 35.5 mm to (218.4, 99.1)
- moved U31 35.5 mm to (231.8, 99.1)
- moved C31 35.5 mm to (234.4, 95.2)
- moved U30 30.4 mm to (245.1, 66.0)
- moved C30 30.4 mm to (247.7, 62.2)
- moved C38 29.3 mm to (304.2, 62.2)
- moved U38 29.3 mm to (301.5, 66.0)
- moved C33 28.3 mm to (264.2, 62.2)
- moved U33 28.3 mm to (261.6, 66.0)
- moved C25 28.1 mm to (207.7, 62.2)
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Connections:
- U25 pad 11: one_count_{12} -> one_count_{15}
- U25 pad 13: one_count_{13} -> one_count_{14}
- U25 pad 15: one_count_{14} -> one_count_{12}
- U25 pad 16: data_{1} -> data_{0}
- U25 pad 17: one_count_{15} -> one_count_{13}
- U25 pad 18: data_{0} -> data_{1}
- U25 pad 2: one_count_{8} -> one_count_{9}
- U25 pad 3: data_{7} -> data_{5}
- U25 pad 4: one_count_{9} -> one_count_{8}
- U25 pad 5: data_{6} -> data_{4}
- U25 pad 7: data_{5} -> data_{6}
- U25 pad 9: data_{4} -> data_{7}
- U28 pad 16: data_{1} -> data_{0}
- U28 pad 18: data_{0} -> data_{1}
- U28 pad 2: one_count_{0} -> one_count_{1}
- U28 pad 4: one_count_{1} -> one_count_{0}
- U30 pad 16: addr_{9} -> addr_{8}
- U30 pad 18: addr_{8} -> addr_{9}
- U30 pad 2: one_count_{8} -> one_count_{9}
- U30 pad 4: one_count_{9} -> one_count_{8}
- U32 pad 16: addr_{1} -> addr_{0}
- U32 pad 18: addr_{0} -> addr_{1}
- U32 pad 2: one_count_{0} -> one_count_{1}
- U32 pad 4: one_count_{1} -> one_count_{0}
- U33 pad 11: two_count_{12} -> two_count_{15}
- U33 pad 13: two_count_{13} -> two_count_{14}
- U33 pad 15: two_count_{14} -> two_count_{12}
- U33 pad 16: data_{1} -> data_{0}
- U33 pad 17: two_count_{15} -> two_count_{13}
- U33 pad 18: data_{0} -> data_{1}
- U33 pad 2: two_count_{8} -> two_count_{9}
- U33 pad 3: data_{7} -> data_{5}
- U33 pad 4: two_count_{9} -> two_count_{8}
- U33 pad 5: data_{6} -> data_{4}
- U33 pad 7: data_{5} -> data_{6}
- U33 pad 9: data_{4} -> data_{7}
- U36 pad 16: data_{1} -> data_{0}
- U36 pad 18: data_{0} -> data_{1}
- U36 pad 2: two_count_{0} -> two_count_{1}
- U36 pad 4: two_count_{1} -> two_count_{0}
- U38 pad 16: addr_{9} -> addr_{8}
- U38 pad 18: addr_{8} -> addr_{9}
- U38 pad 2: two_count_{8} -> two_count_{9}
- U38 pad 4: two_count_{9} -> two_count_{8}
- U40 pad 16: addr_{1} -> addr_{0}
- U40 pad 18: addr_{0} -> addr_{1}
- U40 pad 2: two_count_{0} -> two_count_{1}
- U40 pad 4: two_count_{1} -> two_count_{0}
Routing:
- net +5V: track 637.8 -> 1222.8 mm
- net data_{0}: track 898.1 -> 1158.7 mm, vias 24 -> 36
- net data_{2}: track 811.5 -> 1038.9 mm, vias 24 -> 39
- net ~{write_two_l}: track 0.00 -> 218.1 mm, vias 0 -> 3
- net data_{1}: track 819.7 -> 1012.8 mm, vias 23 -> 35
- net ~{addr_two}: track 0.00 -> 188.0 mm, vias 0 -> 2
- net ~{write_two_h}: track 0.00 -> 186.2 mm, vias 0 -> 2
- net data_{3}: track 768.5 -> 952.9 mm, vias 21 -> 34
- net inc_two: track 0.00 -> 170.6 mm, vias 0 -> 2
- net addr_{3}: track 503.7 -> 673.1 mm, vias 4 -> 6
- net data_{6}: track 745.7 -> 901.7 mm, vias 20 -> 29
- net addr_{2}: track 487.6 -> 643.2 mm, vias 4 -> 6
- net addr_{4}: track 501.3 -> 653.7 mm, vias 4 -> 6
- net ~{read_two_l}: track 0.00 -> 149.8 mm, vias 0 -> 3
- net data_{4}: track 771.8 -> 919.2 mm, vias 23 -> 33
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
Commit message: avançado na otimização do pcb
Parts:
- moved C19 0.08 mm to (176.6, 62.2)
- moved U19 0.08 mm to (174.0, 66.0)
Connections:
- J3 pad 10: rd_addr_1 -> unconnected-(J3-Pin_10-Pad10)
- J3 pad 11: wr_addr_3 -> wr_addr_0
- J3 pad 12: rd_addr_2 -> wr_addr_1
- J3 pad 13: wr_addr_4 -> wr_addr_2
- J3 pad 14: rd_addr_3 -> wr_addr_3
- J3 pad 15: unconnected-(J3-Pin_15-Pad15) -> wr_addr_4
- J3 pad 16: rd_addr_4 -> write_clock
- J3 pad 5: wr_addr_0 -> rd_addr_0
- J3 pad 6: write_clock -> rd_addr_1
- J3 pad 7: wr_addr_1 -> rd_addr_2
- J3 pad 8: rd_addr_0 -> rd_addr_3
- J3 pad 9: wr_addr_2 -> rd_addr_4
Routing:
- net data_{2}: track 1038.9 -> 924.2 mm, vias 39 -> 28
- net data_{3}: track 952.9 -> 841.5 mm, vias 34 -> 23
- net data_{0}: track 1158.7 -> 1086.5 mm, vias 36 -> 32
- net data_{7}: track 877.2 -> 839.8 mm, vias 16 -> 14
- net data_{6}: track 901.7 -> 879.0 mm, vias 29 -> 22
- net rd_addr_4: track 128.6 -> 112.3 mm, vias 2 -> 0
- net data_{1}: track 1012.8 -> 998.6 mm, vias 35 -> 33
- net rd_addr_2: track 123.2 -> 110.2 mm, vias 2 -> 0
- net rd_addr_3: track 125.9 -> 114.3 mm, vias 2 -> 0
- net write_clock: track 146.1 -> 136.2 mm
- net +5V: track 1222.8 -> 1232.5 mm
- net ~{read_marh}: track 170.5 -> 161.9 mm
- net wr_addr_1: track 135.5 -> 127.2 mm, vias 2 -> 0
- net ~{read_marl}: track 206.4 -> 198.6 mm
- net rd_addr_1: track 120.5 -> 113.2 mm, vias 2 -> 0
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