File: pcb_v3/sysbus/sysbus.kicad_pcb (KiCad board)
At the start: 2 copper layers, 297 x 75 mm, 66 parts, among them J1 bus ula 2, J11 bus clu 2, J12 bus clu 3, J19 9V 1A, J2 bus ula 1, J20 VOLTS, J21 AMPS, J22 bus ioc 2, J23 bus ioc 1, J24 bus ioc 3, J26 bus clock, J3 bus rf16 1, J4 bus rf16 2, J5 bus mem 1, J6 bus mem 2, J7 bus clu 1, Q1 BC548, Q2 BC548, SW1 RESET, U1 MC14495P, U10 MC14495P, U11 ADDR N1, U12 DATA N0, U13 MC14495P, U14 RDADDR_LOW, U17 RDADDR_HIGH, U2 ADDR N3, U21 MC14495P, U22 WRADDR_HIGH, U23 WRADDR_LOW, U3 MC14495P, U31 MC14495P, U34 LM7805, U4 ADDR N2, U5 NE555P, U6 MC14495P, U7 DATA N1, U8 MC14495P, U9 ADDR N0

Commit message: refazendo o layout do pcb
Parts:
- removed J22: bus ioc 2, edge_connector:conector 02x08
- removed RN2, RN3: 10K, Resistor_THT:R_Array_SIP9
- moved J24 15.9 mm to (264.2, 42.5)
- moved J4 15.9 mm to (294.6, 42.5)
- moved J11 5.08 mm to (165.1, 53.3)
- moved Q1 1.91 mm to (106.0, 58.4)
- moved Q2 1.27 mm to (111.8, 58.4)
Connections:
- J24 pad 2: unconnected-(J24-Pin_2-Pad2) -> CLOCK
- J24 pad 4: unconnected-(J24-Pin_4-Pad4) -> WRITE_ENABLE
- J24 pad 6: unconnected-(J24-Pin_6-Pad6) -> INT_REQUEST
Routing:
- net ADDR_{5}: track 245.5 -> 48.1 mm, vias 4 -> 2
- net ADDR_{6}: track 247.6 -> 50.7 mm, vias 4 -> 2
- net ADDR_{4}: track 245.4 -> 48.9 mm, vias 4 -> 2
- net ADDR_{7}: track 243.5 -> 47.1 mm, vias 3 -> 2
- net ADDR_{3}: track 223.6 -> 29.7 mm, vias 3 -> 1
- net ADDR_{2}: track 228.5 -> 34.7 mm, vias 3 -> 0
- net ADDR_{0}: track 262.1 -> 82.4 mm, vias 5 -> 0
- net ADDR_{1}: track 260.0 -> 85.5 mm, vias 5 -> 1
- net ADDR_{8}: track 226.5 -> 76.7 mm, vias 3 -> 2
- net ADDR_{9}: track 224.3 -> 77.5 mm, vias 3 -> 2
- net ADDR_{10}: track 229.5 -> 85.8 mm, vias 3 -> 2
- net ADDR_{11}: track 221.7 -> 81.0 mm, vias 3 -> 2
- net ADDR_{12}: track 233.4 -> 95.3 mm, vias 3 -> 2
- net ADDR_{13}: track 231.4 -> 95.3 mm, vias 3 -> 2
- net ADDR_{14}: track 237.1 -> 102.9 mm, vias 3 -> 2
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
Commit message: avançando no layot v3
Parts:
- moved R12 4.96 mm to (135.9, 53.3), turned to 180 degrees
Routing:
- net WR_ADDR_1: track 228.8 -> 235.7 mm
- net WR_ADDR_4: track 246.2 -> 252.0 mm
- net RD_ADDR_3: track 216.3 -> 220.4 mm, vias 4 -> 3
- net WR_ADDR_0: track 223.2 -> 227.2 mm
- net RD_ADDR_2: track 211.5 -> 215.5 mm, vias 4 -> 3
- net Net-(U13-a): track 24.2 -> 26.8 mm, vias 1 -> 0
- net RD_ADDR_1: track 198.3 -> 195.7 mm, vias 4 -> 3
- net ULA_ENABLE: track 51.5 -> 49.0 mm, vias 2 -> 1
- net Net-(R12-Pad1): track 46.8 -> 49.3 mm
- net RD_ADDR_0: track 187.0 -> 188.2 mm, vias 4 -> 3
- net WR_ADDR_2: track 238.0 -> 237.3 mm, vias 5 -> 4
- net WR_ADDR_3: vias 6 -> 5
- net WRITE_ENABLE: vias 3 -> 2
- net ~{UC_pcia_swap}: vias 1 -> 0
- net MEMORY_READ: vias 2 -> 1
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Other:
- board text added: "Rev.3A julho/2026"
- board text removed: "Rev.3A junho/2026"

Commit message: preparação para produção das pcbs
Other:
- board text added: "Rev.3-A julho/2026"
- board text removed: "Rev.3A julho/2026"
Changed lines of the file:
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@@
 		(tenting front back)
 		(pcbplotparams
-			(layerselection 0x00000000_00000000_55555555_5755f5ff)
+			(layerselection 0x00000000_00000000_55555555_575555ff)
 			(plot_on_all_layers_selection 0x00000000_00000000_00000000_00000000)
 			(disableapertmacros no)
@@
 			(outputformat 1)
 			(mirror no)
-			(drillshape 1)
+			(drillshape 0)
 			(scaleselection 1)
-			(outputdirectory "")
+			(outputdirectory "plot")
 		)
 	)
@@
 		)
 	)
-	(gr_text "Rev.3A julho/2026"
+	(gr_text "Rev.3-A julho/2026"
 		(at 316.23 54.61 90)
 		(layer "F.SilkS")
