File: pcb_v3/clu/clu.kicad_pcb (KiCad board)
At the start: 2 copper layers, 160.7 x 210 mm, 86 parts, among them J1 bus clu 1, J11 UCODE 1, J12 UCODE 2, J13 UCODE 3, J14 UCODE 4, J15 UCODE 5, J16 UCODE 6, J18 UCODE INT, J2 bus clu 2, J3 bus clu 3, J4 UCODE RESET, J5 UCODE 7, J7 UCODE 0, SW1 SW_DIP_read_mem_const, SW3 SW_DIP_mem_pc, SW6 SW_DIP_pc, U1 74LS193, U10 MC14495P, U11 IR_HIGH, U12 74LS574, U13 74LS244, U15 74LS244, U16 74LS86, U17 74LS157, U19 74LS04, U2 74LS138, U20 74LS08, U24 74LS86, U25 74LS125, U26 74LS32, U27 74LS08, U28 74LS74, U29 74LS74, U3 74LS157, U30 74LS138, U31 MC14495P, U32 74LS138, U4 74LS02, U6 74LS157, U7 74LS157, U8 74LS574, U9 IR_LOW

Commit message: .
Changed lines of the file:
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@@
 	)
 	(gr_rect
-		(start 286.385 18.0975)
-		(end 296.545 133.0325)
+		(start 224.155 49.53)
+		(end 236.855 148.59)
 		(stroke
 			(width 0.1)
+			(type solid)
+		)
+		(fill no)
+		(layer "F.SilkS")
+	)
+	(gr_rect
+		(start 238.125 49.53)
+		(end 250.825 152.4)
+		(stroke
+			(width 0.1)
+			(type solid)
+		)
+		(fill no)
+		(layer "F.SilkS")
+	)
+	(gr_rect
+		(start 252.095 49.53)
+		(end 264.795 152.4)
+		(stroke
+			(width 0.1)
+			(type solid)
+		)
+		(fill no)
+		(layer "F.SilkS")
+	)
+	(gr_rect
+		(start 266.065 49.53)
+		(end 278.765 152.4)
+		(stroke
+			(width 0.1)
+			(type solid)
+		)
+		(fill no)
+		(layer "F.SilkS")
+	)
+	(gr_rect
+		(start 280.035 49.53)
+		(end 292.735 152.4)
+		(stroke
+			(width 0.1)
+			(type solid)
+		)
+		(fill no)
+		(layer "F.SilkS")
+	)
+	(gr_rect
+		(start 294.005 49.53)
+		(end 306.705 152.4)
+		(stroke
+			(width 0.1)
+			(type solid)
+		)
+		(fill no)
+		(layer "F.SilkS")
+	)
+	(gr_rect
+		(start 307.975 49.53)
+		(end 320.675 152.4)
+		(stroke
+			(width 0.1)
+			(type solid)
+		)
+		(fill no)
+		(layer "F.SilkS")
+	)
+	(gr_rect
+		(start 321.945 49.53)
+		(end 334.645 152.4)
+		(stroke
+			(width 0.1)
+			(type solid)
+		)
+		(fill no)
+		(layer "F.SilkS")
+	)
+	(gr_rect
+		(start 335.915 49.53)
+		(end 348.615 152.4)
+		(stroke
+			(width 0.1)
+			(type solid)
+		)
+		(fill no)
+		(layer "F.SilkS")
+	)
+	(gr_rect
+		(start 349.885 49.53)
+		(end 362.585 152.4)
+		(stroke
+			(width 0.1)

Commit message: layout usando a ROM de opcode na horizontal
Parts:
- added C11: 100nF, Capacitor_THT:C_Disc_D5.1mm_W3.2mm_P5.00mm, F.Cu at (62.9, 31.1)
- added C14: 100nF, Capacitor_THT:C_Disc_D5.1mm_W3.2mm_P5.00mm, F.Cu at (76.9, 31.1)
- added C18: 100nF, Capacitor_THT:C_Disc_D5.1mm_W3.2mm_P5.00mm, F.Cu at (90.9, 31.1)
- added C21: 100nF, Capacitor_THT:C_Disc_D5.1mm_W3.2mm_P5.00mm, F.Cu at (104.9, 31.1)
- added C22: 100nF, Capacitor_THT:C_Disc_D5.1mm_W3.2mm_P5.00mm, F.Cu at (118.8, 31.1)
- added C23: 100nF, Capacitor_THT:C_Disc_D5.1mm_W3.2mm_P5.00mm, F.Cu at (132.8, 31.1)
- added C33: 100nF, Capacitor_THT:C_Disc_D5.1mm_W3.2mm_P5.00mm, F.Cu at (146.8, 31.1)
- added C5: 100nF, Capacitor_THT:C_Disc_D5.1mm_W3.2mm_P5.00mm, F.Cu at (35.0, 31.1)
- added C9: 100nF, Capacitor_THT:C_Disc_D5.1mm_W3.2mm_P5.00mm, F.Cu at (49.0, 31.1)
- added J10: Conn_01x07, Connector_PinHeader_2.54mm:PinHeader_1x07_P2.54mm_Vertical, F.Cu at (137.2, 119.4)
- added J17: Conn_01x07, Connector_PinHeader_2.54mm:PinHeader_1x07_P2.54mm_Vertical, F.Cu at (102.9, 119.4)
- added J19: Conn_01x07, Connector_PinHeader_2.54mm:PinHeader_1x07_P2.54mm_Vertical, F.Cu at (95.2, 119.4)
- added J20: Conn_01x07, Connector_PinHeader_2.54mm:PinHeader_1x07_P2.54mm_Vertical, F.Cu at (88.9, 119.4)
- added J21: Conn_01x03, Connector_PinHeader_2.54mm:PinHeader_1x03_P2.54mm_Vertical, F.Cu at (108.6, 26.0)
- added J22: Conn_01x07, Connector_PinHeader_2.54mm:PinHeader_1x07_P2.54mm_Vertical, F.Cu at (81.3, 119.4)
- added J23: Conn_01x07, Connector_PinHeader_2.54mm:PinHeader_1x07_P2.54mm_Vertical, F.Cu at (74.9, 119.4)
- added J24: Conn_01x03, Connector_PinHeader_2.54mm:PinHeader_1x03_P2.54mm_Vertical, F.Cu at (122.6, 26.0)
- added J25: Conn_01x07, Connector_PinHeader_2.54mm:PinHeader_1x07_P2.54mm_Vertical, F.Cu at (67.3, 119.4)
- added J26: Conn_01x07, Connector_PinHeader_2.54mm:PinHeader_1x07_P2.54mm_Vertical, F.Cu at (61.0, 119.4)
- added J27: Conn_01x03, Connector_PinHeader_2.54mm:PinHeader_1x03_P2.54mm_Vertical, F.Cu at (136.5, 26.0)
- added J28: Conn_01x07, Connector_PinHeader_2.54mm:PinHeader_1x07_P2.54mm_Vertical, F.Cu at (53.3, 119.4)
- added J29: Conn_01x07, Connector_PinHeader_2.54mm:PinHeader_1x07_P2.54mm_Vertical, F.Cu at (39.4, 119.4)
- added J30: Conn_01x07, Connector_PinHeader_2.54mm:PinHeader_1x07_P2.54mm_Vertical, F.Cu at (33.0, 119.4)
- added J31: Conn_01x07, Connector_PinHeader_2.54mm:PinHeader_1x07_P2.54mm_Vertical, F.Cu at (47.0, 119.4)
- added J32: Conn_01x03, Connector_PinHeader_2.54mm:PinHeader_1x03_P2.54mm_Vertical, F.Cu at (150.5, 26.0)
- added J33: Conn_01x03, Connector_PinHeader_2.54mm:PinHeader_1x03_P2.54mm_Vertical, F.Cu at (164.5, 26.0)
- added J6: Conn_01x07, Connector_PinHeader_2.54mm:PinHeader_1x07_P2.54mm_Vertical, F.Cu at (151.1, 119.4)
- added J8: Conn_01x07, Connector_PinHeader_2.54mm:PinHeader_1x07_P2.54mm_Vertical, F.Cu at (144.8, 119.4)
- added J9: Conn_01x03, Connector_PinHeader_2.54mm:PinHeader_1x03_P2.54mm_Vertical, F.Cu at (38.7, 26.0)
- added U14: 74LS32, Package_DIP:DIP-14_W7.62mm, F.Cu at (46.4, 34.9)
- added U18: 74LS32, Package_DIP:DIP-14_W7.62mm, F.Cu at (60.3, 34.9)
- added U21: 74LS32, Package_DIP:DIP-14_W7.62mm, F.Cu at (74.3, 34.9)
- added U22: 74LS32, Package_DIP:DIP-14_W7.62mm, F.Cu at (88.3, 34.9)
- added U23: 74LS32, Package_DIP:DIP-14_W7.62mm, F.Cu at (102.2, 34.9)
- added U33: 74LS32, Package_DIP:DIP-14_W7.62mm, F.Cu at (116.2, 34.9)
- added U34: 74LS32, Package_DIP:DIP-14_W7.62mm, F.Cu at (130.2, 34.9)
- added U35: 74LS32, Package_DIP:DIP-14_W7.62mm, F.Cu at (144.1, 34.9)
- added U5: 74LS32, Package_DIP:DIP-14_W7.62mm, F.Cu at (32.4, 34.9)
- J11: value UCODE 1 -> Conn_01x07; footprint edge_connector:male-edge-connector-28 -> Connector_PinHeader_2.54mm:PinHeader_1x07_P2.54mm_Vertical
- J12: value UCODE 2 -> Conn_01x03; footprint edge_connector:male-edge-connector-28 -> Connector_PinHeader_2.54mm:PinHeader_1x03_P2.54mm_Vertical
- J13: value UCODE 3 -> Conn_01x07; footprint edge_connector:male-edge-connector-28 -> Connector_PinHeader_2.54mm:PinHeader_1x07_P2.54mm_Vertical
- J14: value UCODE 4 -> Conn_01x07; footprint edge_connector:male-edge-connector-28 -> Connector_PinHeader_2.54mm:PinHeader_1x07_P2.54mm_Vertical
- J15: value UCODE 5 -> Conn_01x03; footprint edge_connector:male-edge-connector-28 -> Connector_PinHeader_2.54mm:PinHeader_1x03_P2.54mm_Vertical
- J16: value UCODE 6 -> Conn_01x07; footprint edge_connector:male-edge-connector-28 -> Connector_PinHeader_2.54mm:PinHeader_1x07_P2.54mm_Vertical
- J18: value UCODE INT -> Conn_01x03; footprint edge_connector:male-edge-connector-28 -> Connector_PinHeader_2.54mm:PinHeader_1x03_P2.54mm_Vertical
- J4: value UCODE RESET -> Conn_01x07; footprint edge_connector:male-edge-connector-28 -> Connector_PinHeader_2.54mm:PinHeader_1x07_P2.54mm_Vertical
- J5: value UCODE 7 -> Conn_01x07; footprint edge_connector:male-edge-connector-28 -> Connector_PinHeader_2.54mm:PinHeader_1x07_P2.54mm_Vertical
- J7: value UCODE 0 -> Conn_01x03; footprint edge_connector:male-edge-connector-28 -> Connector_PinHeader_2.54mm:PinHeader_1x03_P2.54mm_Vertical
- moved J11 120.8 mm to (130.8, 119.4), turned to 180 degrees
- moved R12 100.0 mm to (147.3, 128.9)
- moved J13 99.7 mm to (123.2, 119.4), turned to 180 degrees
- moved J5 92.3 mm to (158.8, 119.4), turned to 180 degrees
- moved J14 90.8 mm to (116.8, 119.4), turned to 180 degrees
- moved C29 88.3 mm to (101.7, 165.7)
- moved U29 88.3 mm to (99.1, 169.5)
- moved J4 86.1 mm to (165.1, 119.4), turned to 180 degrees
- moved J16 83.8 mm to (109.2, 119.4), turned to 180 degrees
- moved RN3 39.6 mm to (158.8, 87.0), turned to -90 degrees
- moved J18 39.3 mm to (94.6, 26.0), turned to -90 degrees
- moved C25 31.2 mm to (146.8, 59.1)
- moved U25 31.2 mm to (144.1, 62.9)
- moved C4 30.2 mm to (132.8, 59.1)
- moved U4 30.2 mm to (130.2, 62.9)
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Connections:
- J11 pad 1: +5V -> ~{UC_write_to_pc}
- J11 pad 2: unconnected-(J11-Pin_2-Pad2) -> ~{UC_write_enable}
- J11 pad 3: unconnected-(J11-Pin_3-Pad3) -> ~{UC_int_ready}
- J11 pad 4: unconnected-(J11-Pin_4-Pad4) -> ~{UC_read_mem_const}
- J11 pad 5: unconnected-(J11-Pin_5-Pad5) -> ~{UC_A}
- J11 pad 6: ~{UC_extended_opcode} -> ~{UC_read_addr_src_reg}
- J11 pad 7: unconnected-(J11-Pin_7-Pad7) -> ~{UC_pcia_swap}
- J12 pad 1: +5V -> Net-(J12-Pin_1)
- J12 pad 2: unconnected-(J12-Pin_2-Pad2) -> Net-(J12-Pin_2)
- J12 pad 3: unconnected-(J12-Pin_3-Pad3) -> Net-(J12-Pin_3)
- J13 pad 1: +5V -> ~{UC_disable_int}
- J13 pad 2: unconnected-(J13-Pin_2-Pad2) -> ~{UC_extended_opcode}
- J13 pad 3: unconnected-(J13-Pin_3-Pad3) -> ~{UC_ula_enable}
- J13 pad 4: unconnected-(J13-Pin_4-Pad4) -> ~{UC_save_src_reg}
- J13 pad 5: unconnected-(J13-Pin_5-Pad5) -> ~{UC_restart_cycle}
- J13 pad 6: ~{UC_extended_opcode} -> ~{UC_save_cond_reg}
- J13 pad 7: unconnected-(J13-Pin_7-Pad7) -> ~{UC_clear_cond_reg}
- J14 pad 1: +5V -> ~{UC_write_to_pc}
- J14 pad 2: unconnected-(J14-Pin_2-Pad2) -> ~{UC_write_enable}
- J14 pad 3: unconnected-(J14-Pin_3-Pad3) -> ~{UC_int_ready}
- J14 pad 4: unconnected-(J14-Pin_4-Pad4) -> ~{UC_read_mem_const}
- J14 pad 5: unconnected-(J14-Pin_5-Pad5) -> ~{UC_A}
- J14 pad 6: ~{UC_extended_opcode} -> ~{UC_read_addr_src_reg}
- J14 pad 7: unconnected-(J14-Pin_7-Pad7) -> ~{UC_pcia_swap}
- J15 pad 1: +5V -> Net-(J15-Pin_1)
- J15 pad 2: unconnected-(J15-Pin_2-Pad2) -> Net-(J15-Pin_2)
- J15 pad 3: unconnected-(J15-Pin_3-Pad3) -> Net-(J15-Pin_3)
- J16 pad 1: +5V -> ~{UC_disable_int}
- J16 pad 2: unconnected-(J16-Pin_2-Pad2) -> ~{UC_extended_opcode}
- J16 pad 3: unconnected-(J16-Pin_3-Pad3) -> ~{UC_ula_enable}
- J16 pad 4: unconnected-(J16-Pin_4-Pad4) -> ~{UC_save_src_reg}
- J16 pad 5: unconnected-(J16-Pin_5-Pad5) -> ~{UC_restart_cycle}
- J16 pad 6: ~{UC_extended_opcode} -> ~{UC_save_cond_reg}
- J16 pad 7: unconnected-(J16-Pin_7-Pad7) -> ~{UC_clear_cond_reg}
- J18 pad 1: +5V -> Net-(J18-Pin_1)
- J18 pad 2: unconnected-(J18-Pin_2-Pad2) -> Net-(J18-Pin_2)
- J18 pad 3: unconnected-(J18-Pin_3-Pad3) -> Net-(J18-Pin_3)
- J4 pad 1: +5V -> ~{UC_disable_int}
- J4 pad 2: unconnected-(J4-Pin_2-Pad2) -> ~{UC_extended_opcode}
- J4 pad 3: unconnected-(J4-Pin_3-Pad3) -> ~{UC_ula_enable}
- J4 pad 4: unconnected-(J4-Pin_4-Pad4) -> ~{UC_save_src_reg}
- J4 pad 5: unconnected-(J4-Pin_5-Pad5) -> ~{UC_restart_cycle}
- J4 pad 6: ~{UC_extended_opcode} -> ~{UC_save_cond_reg}
- J4 pad 7: unconnected-(J4-Pin_7-Pad7) -> ~{UC_clear_cond_reg}
- J5 pad 1: +5V -> ~{UC_write_to_pc}
- J5 pad 2: unconnected-(J5-Pin_2-Pad2) -> ~{UC_write_enable}
- J5 pad 3: unconnected-(J5-Pin_3-Pad3) -> ~{UC_int_ready}
- J5 pad 4: unconnected-(J5-Pin_4-Pad4) -> ~{UC_read_mem_const}
- J5 pad 5: unconnected-(J5-Pin_5-Pad5) -> ~{UC_A}
- J5 pad 6: ~{UC_extended_opcode} -> ~{UC_read_addr_src_reg}
- J5 pad 7: unconnected-(J5-Pin_7-Pad7) -> ~{UC_pcia_swap}
- J7 pad 1: +5V -> Net-(J7-Pin_1)
- J7 pad 2: unconnected-(J7-Pin_2-Pad2) -> Net-(J7-Pin_2)
- J7 pad 3: unconnected-(J7-Pin_3-Pad3) -> Net-(J7-Pin_3)
- RN3 pad 2: ~{UC_int_ready} -> ~{UC_read_mem_const}
- RN3 pad 3: ~{UC_write_enable} -> ~{UC_A}
- RN3 pad 4: ~{UC_extended_opcode} -> ~{UC_read_addr_src_reg}
- RN3 pad 5: ~{UC_save_cond_reg} -> ~{UC_pcia_swap}
- RN4 pad 2: ~{UC_A} -> unconnected-(RN4-R1-Pad2)
- RN4 pad 3: ~{UC_read_mem_const} -> ~{UC_write_to_pc}
- RN4 pad 4: ~{UC_pcia_swap} -> ~{UC_write_enable}
- RN4 pad 5: ~{UC_ula_enable} -> ~{UC_int_ready}
- RN5 pad 2: ~{UC_restart_cycle} -> ~{UC_save_src_reg}
- RN5 pad 3: ~{UC_clear_cond_reg} -> ~{UC_restart_cycle}
- RN5 pad 4: ~{UC_disable_int} -> ~{UC_save_cond_reg}
- RN5 pad 5: ~{UC_save_src_reg} -> ~{UC_clear_cond_reg}
- RN7 pad 3: unconnected-(RN7-R2-Pad3) -> ~{UC_disable_int}
- RN7 pad 4: ~{UC_write_to_pc} -> ~{UC_extended_opcode}
- RN7 pad 5: ~{UC_read_addr_src_reg} -> ~{UC_ula_enable}
- U16 pad 10: INS_{0} -> ~{low_cycle}
- U16 pad 9: ~{low_cycle} -> INS_{0}
- U19 pad 1: +5V -> ~{UC_save_cond_reg}
- U19 pad 10: Net-(U12-Cp) -> unconnected-(U19-Pad10)
- U19 pad 11: ~{UC_save_src_reg} -> +5V
- U19 pad 2: unconnected-(U19-Pad2) -> Net-(U28A-C)
- U19 pad 3: ~{UC_save_cond_reg} -> fetch_clock
- U19 pad 4: Net-(U28A-C) -> ~{fetch_clock}
- U19 pad 5: fetch_clock -> ~{UC_save_src_reg}
- U19 pad 6: ~{fetch_clock} -> Net-(U12-Cp)
Routing:
- net +5V: track 1190.6 -> 851.3 mm, vias 2 -> 1
- net INS_{7}: track 302.5 -> 21.1 mm, vias 3 -> 0
- net INS_{6}: track 302.4 -> 23.9 mm, vias 2 -> 0
- net INS_{5}: track 292.6 -> 26.7 mm, vias 5 -> 0
- net INT_REQUEST: track 248.5 -> 0.00 mm, vias 3 -> 0
- net INS_{4}: track 284.8 -> 66.1 mm, vias 4 -> 3
- net INS_{1}: track 274.6 -> 67.6 mm, vias 7 -> 2
- net INS_{2}: track 254.1 -> 61.6 mm, vias 7 -> 2
- net RD_ADDR_4: track 183.3 -> 0.00 mm, vias 4 -> 0
- net RD_ADDR_3: track 182.1 -> 0.00 mm, vias 5 -> 0
- net INS_{3}: track 248.1 -> 68.5 mm, vias 7 -> 2
- net RD_ADDR_2: track 171.2 -> 0.00 mm, vias 3 -> 0
- net RD_ADDR_1: track 170.7 -> 0.00 mm, vias 5 -> 0
- net ~{UC_pcia_swap}: track 299.7 -> 142.2 mm, vias 4 -> 0
- net INT_MASK_FLAG: track 150.8 -> 0.00 mm, vias 5 -> 0
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
Commit message: avançando no novo layout
Parts:
- moved U29 19.1 mm to (99.1, 188.6)
- moved C29 19.0 mm to (101.7, 184.8)
- moved C7 17.3 mm to (151.2, 182.2)
- moved U7 17.3 mm to (148.6, 186.1)
- moved U17 16.5 mm to (82.5, 186.1)
- moved C17 16.5 mm to (85.2, 182.2)
- moved C8 16.5 mm to (167.7, 177.2)
- moved U8 16.5 mm to (165.1, 181.0)
- moved D5 10.8 mm to (112.4, 182.2), turned to 90 degrees
- moved C6 5.08 mm to (134.7, 182.2)
- moved U6 5.08 mm to (132.1, 186.1)
- moved C30 5.08 mm to (118.2, 182.2)
- moved U30 5.08 mm to (115.6, 186.1)
- moved C13 0.16 mm to (52.1, 165.7)
- moved C15 0.16 mm to (68.7, 165.7)
Routing:
- net +5V: track 851.3 -> 1093.2 mm, vias 1 -> 2
- net ~{fetch_cycle}: track 179.3 -> 346.0 mm, vias 1 -> 4
- net INS_{6}: track 23.9 -> 185.0 mm, vias 0 -> 1
- net INS_{7}: track 21.1 -> 180.1 mm, vias 0 -> 1
- net INS_{2}: track 61.6 -> 215.6 mm, vias 2 -> 6
- net INS_{5}: track 26.7 -> 168.7 mm, vias 0 -> 2
- net INS_{4}: track 66.1 -> 188.3 mm, vias 3 -> 4
- net INS_{1}: track 67.6 -> 186.6 mm, vias 2 -> 4
- net ~{condition_true}: track 127.1 -> 239.7 mm, vias 1 -> 3
- net INS_{3}: track 68.5 -> 174.7 mm, vias 2 -> 3
- net ~{low_cycle}: track 351.5 -> 455.5 mm, vias 3 -> 5
- net INS_{0}: track 219.9 -> 317.1 mm, vias 2 -> 5
- net ~{UC_pclr_swap}: track 0.00 -> 95.3 mm, vias 0 -> 1
- net INT_MASK_FLAG: track 0.00 -> 92.8 mm, vias 0 -> 2
- net RD_ADDR_4: track 0.00 -> 91.7 mm, vias 0 -> 1
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
Commit message: conclusão da primeira fase de layout
Routing:
- net INT_REQUEST: track 12.1 -> 182.6 mm, vias 1 -> 6
- net INS_{7}: track 180.1 -> 337.6 mm, vias 1 -> 5
- net INS_{6}: track 185.0 -> 339.1 mm, vias 1 -> 5
- net INS_{5}: track 168.7 -> 319.7 mm, vias 2 -> 6
- net +5V: track 1093.2 -> 1218.8 mm, vias 2 -> 3
- net RD_ADDR_2: track 68.1 -> 181.1 mm, vias 0 -> 4
- net WR_ADDR_2: track 31.2 -> 140.4 mm, vias 0 -> 3
- net WR_ADDR_3: track 34.7 -> 139.2 mm, vias 0 -> 3
- net WR_ADDR_1: track 27.8 -> 131.7 mm, vias 0 -> 3
- net ~{enable_wr_addr}: track 0.00 -> 102.9 mm, vias 0 -> 4
- net RD_ADDR_3: track 78.0 -> 180.1 mm, vias 1 -> 4
- net RD_ADDR_1: track 75.3 -> 174.0 mm, vias 1 -> 4
- net ~{UC_write_to_pc}: track 179.1 -> 275.0 mm, vias 0 -> 2
- net RD_ADDR_0: track 35.8 -> 131.2 mm, vias 0 -> 3
- net OVERFLOW_FLAG: track 1.80 -> 95.7 mm
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