File: pcb_v3/clu/clu.kicad_sch (KiCad schematic)
At the start: 86 parts, among them J1 bus clu 1, J11 UCODE 1, J12 UCODE 2, J13 UCODE 3, J14 UCODE 4, J15 UCODE 5, J16 UCODE 6, J18 UCODE INT, J2 bus clu 2, J3 bus clu 3, J4 UCODE RESET, J5 UCODE 7, J7 UCODE 0, SW1 SW_DIP_read_mem_const, SW3 SW_DIP_mem_pc, SW6 SW_DIP_pc, U1 74LS193, U10 MC14495P, U11 IR_HIGH, U12 74LS574, U13 74LS244, U15 74LS244, U16 74LS86, U17 74LS157, U19 74LS04, U2 74LS138, U20 74LS08, U24 74LS86, U25 74LS125, U26 74LS32, U27 74LS08, U28 74LS74, U29 74LS74, U3 74LS157, U30 74LS138, U31 MC14495P, U32 74LS138, U4 74LS02, U6 74LS157, U7 74LS157, U8 74LS574, U9 IR_LOW

Commit message: layout usando a ROM de opcode na horizontal
Parts:
- removed J11: UCODE 1, edge_connector:male-edge-connector-28, symbol Connector_Generic:Conn_02x14_Top_Bottom
- removed J12: UCODE 2, edge_connector:male-edge-connector-28, symbol Connector_Generic:Conn_02x14_Top_Bottom
- removed J13: UCODE 3, edge_connector:male-edge-connector-28, symbol Connector_Generic:Conn_02x14_Top_Bottom
- removed J14: UCODE 4, edge_connector:male-edge-connector-28, symbol Connector_Generic:Conn_02x14_Top_Bottom
- removed J15: UCODE 5, edge_connector:male-edge-connector-28, symbol Connector_Generic:Conn_02x14_Top_Bottom
- removed J16: UCODE 6, edge_connector:male-edge-connector-28, symbol Connector_Generic:Conn_02x14_Top_Bottom
- removed J18: UCODE INT, edge_connector:male-edge-connector-28, symbol Connector_Generic:Conn_02x14_Top_Bottom
- removed J4: UCODE RESET, edge_connector:male-edge-connector-28, symbol Connector_Generic:Conn_02x14_Top_Bottom
- removed J5: UCODE 7, edge_connector:male-edge-connector-28, symbol Connector_Generic:Conn_02x14_Top_Bottom
- removed J7: UCODE 0, edge_connector:male-edge-connector-28, symbol Connector_Generic:Conn_02x14_Top_Bottom
- added C11, C14, C18, C21, C22, C23, C33, C5, C9: 100nF, Capacitor_THT:C_Disc_D5.1mm_W3.2mm_P5.00mm, symbol Device:C
- added J10, J11, J13, J14, J16, J17, J19, J20, J22, J23, J25, J26, J28, J29, J30, J31, J4, J5, J6, J8: Conn_01x07, Connector_PinHeader_2.54mm:PinHeader_1x07_P2.54mm_Vertical, symbol Connector_Generic:Conn_01x07
- added J12, J15, J18, J21, J24, J27, J32, J33, J7, J9: Conn_01x03, Connector_PinHeader_2.54mm:PinHeader_1x03_P2.54mm_Vertical, symbol Connector_Generic:Conn_01x03
- added U14, U18, U21, U22, U23, U33, U34, U35, U5: 74LS32, Package_DIP:DIP-14_W7.62mm, symbol 74xx:74LS32
Connections:
- net +5V: now also U19.11, C11.2, C14.2, C18.2, C21.2, C22.2, C23.2, C33.2, C5.2, C9.2, U14.10, U14.14 (VCC), U14.9, U18.10, U18.14 (VCC), U18.9, U21.10, U21.14 (VCC), U21.9, U22.10, U22.14 (VCC), U22.9, U23.10, U23.14 (VCC), U23.9, U33.10, U33.14 (VCC), U33.9, U34.10, U34.14 (VCC), U34.9, U35.10, U35.14 (VCC), U35.9, U5.10, U5.14 (VCC), U5.9; no longer U19.1
- net GND: now also C11.1, C14.1, C18.1, C21.1, C22.1, C23.1, C33.1, C5.1, C9.1, U14.7 (GND), U18.7 (GND), U21.7 (GND), U22.7 (GND), U23.7 (GND), U33.7 (GND), U34.7 (GND), U35.7 (GND), U5.7 (GND)
- net INS_{0}: now also U16.9; no longer U16.10
- net fetch_clock: now also U19.3; no longer U19.5
- net ~{UC_A}: now also RN3.3 (R2), J11.5 (Pin_5), J14.5 (Pin_5), J17.5 (Pin_5), J20.5 (Pin_5), J23.5 (Pin_5), J26.5 (Pin_5), J30.5 (Pin_5), J31.5 (Pin_5), J5.5 (Pin_5), J8.5 (Pin_5); no longer RN4.2 (R1)
- net ~{UC_clear_cond_reg}: now also RN5.5 (R4), J10.7 (Pin_7), J13.7 (Pin_7), J16.7 (Pin_7), J19.7 (Pin_7), J22.7 (Pin_7), J25.7 (Pin_7), J28.7 (Pin_7), J29.7 (Pin_7), J4.7 (Pin_7), J6.7 (Pin_7); no longer RN5.3 (R2)
- net ~{UC_disable_int}: now also RN7.3 (R2), J10.1 (Pin_1), J13.1 (Pin_1), J16.1 (Pin_1), J19.1 (Pin_1), J22.1 (Pin_1), J25.1 (Pin_1), J28.1 (Pin_1), J29.1 (Pin_1), J4.1 (Pin_1), J6.1 (Pin_1); no longer RN5.4 (R3)
- net ~{UC_extended_opcode}: now also RN7.4 (R3), J10.2 (Pin_2), J13.2 (Pin_2), J16.2 (Pin_2), J19.2 (Pin_2), J22.2 (Pin_2), J25.2 (Pin_2), J28.2 (Pin_2), J29.2 (Pin_2), J4.2 (Pin_2), J6.2 (Pin_2); no longer RN3.4 (R3)
- net ~{UC_int_ready}: now also RN4.5 (R4), J11.3 (Pin_3), J14.3 (Pin_3), J17.3 (Pin_3), J20.3 (Pin_3), J23.3 (Pin_3), J26.3 (Pin_3), J30.3 (Pin_3), J31.3 (Pin_3), J5.3 (Pin_3), J8.3 (Pin_3); no longer RN3.2 (R1)
- net ~{UC_pcia_swap}: now also RN3.5 (R4), J11.7 (Pin_7), J14.7 (Pin_7), J17.7 (Pin_7), J20.7 (Pin_7), J23.7 (Pin_7), J26.7 (Pin_7), J30.7 (Pin_7), J31.7 (Pin_7), J5.7 (Pin_7), J8.7 (Pin_7); no longer RN4.4 (R3)
- net ~{UC_read_addr_src_reg}: now also RN3.4 (R3), J11.6 (Pin_6), J14.6 (Pin_6), J17.6 (Pin_6), J20.6 (Pin_6), J23.6 (Pin_6), J26.6 (Pin_6), J30.6 (Pin_6), J31.6 (Pin_6), J5.6 (Pin_6), J8.6 (Pin_6); no longer RN7.5 (R4)
- net ~{UC_read_mem_const}: now also RN3.2 (R1), J11.4 (Pin_4), J14.4 (Pin_4), J17.4 (Pin_4), J20.4 (Pin_4), J23.4 (Pin_4), J26.4 (Pin_4), J30.4 (Pin_4), J31.4 (Pin_4), J5.4 (Pin_4), J8.4 (Pin_4); no longer RN4.3 (R2)
- net ~{UC_restart_cycle}: now also RN5.3 (R2), J10.5 (Pin_5), J13.5 (Pin_5), J16.5 (Pin_5), J19.5 (Pin_5), J22.5 (Pin_5), J25.5 (Pin_5), J28.5 (Pin_5), J29.5 (Pin_5), J4.5 (Pin_5), J6.5 (Pin_5); no longer RN5.2 (R1)
- net ~{UC_save_cond_reg}: now also RN5.4 (R3), U19.1, J10.6 (Pin_6), J13.6 (Pin_6), J16.6 (Pin_6), J19.6 (Pin_6), J22.6 (Pin_6), J25.6 (Pin_6), J28.6 (Pin_6), J29.6 (Pin_6), J4.6 (Pin_6), J6.6 (Pin_6); no longer RN3.5 (R4), U19.3
- net ~{UC_save_src_reg}: now also RN5.2 (R1), U19.5, J10.4 (Pin_4), J13.4 (Pin_4), J16.4 (Pin_4), J19.4 (Pin_4), J22.4 (Pin_4), J25.4 (Pin_4), J28.4 (Pin_4), J29.4 (Pin_4), J4.4 (Pin_4), J6.4 (Pin_4); no longer RN5.5 (R4), U19.11
- net ~{UC_ula_enable}: now also RN7.5 (R4), J10.3 (Pin_3), J13.3 (Pin_3), J16.3 (Pin_3), J19.3 (Pin_3), J22.3 (Pin_3), J25.3 (Pin_3), J28.3 (Pin_3), J29.3 (Pin_3), J4.3 (Pin_3), J6.3 (Pin_3); no longer RN4.5 (R4)
- net ~{UC_write_enable}: now also RN4.4 (R3), J11.2 (Pin_2), J14.2 (Pin_2), J17.2 (Pin_2), J20.2 (Pin_2), J23.2 (Pin_2), J26.2 (Pin_2), J30.2 (Pin_2), J31.2 (Pin_2), J5.2 (Pin_2), J8.2 (Pin_2); no longer RN3.3 (R2)
- net ~{UC_write_to_pc}: now also RN4.3 (R2), J11.1 (Pin_1), J14.1 (Pin_1), J17.1 (Pin_1), J20.1 (Pin_1), J23.1 (Pin_1), J26.1 (Pin_1), J30.1 (Pin_1), J31.1 (Pin_1), J5.1 (Pin_1), J8.1 (Pin_1); no longer RN7.4 (R3)
- net ~{fetch_clock}: now also U19.4, U14.12, U18.12, U21.12, U22.12, U23.12, U33.12, U34.12, U35.12, U5.12; no longer U19.6
- net ~{high_cycle}: now also U14.4, U18.4, U21.4, U22.4, U23.4, U33.4, U34.4, U35.4, U5.4
- net ~{low_cycle}: now also U16.10, U14.1, U18.1, U21.1, U22.1, U23.1, U33.1, U34.1, U35.1, U5.1; no longer U16.9
- net ~{reset_high_cycle}: now also J33.3 (Pin_3)
- net ~{reset_low_cycle}: now also J33.2 (Pin_2)
- net ~{reset_sync}: now also J33.1 (Pin_1)
- net ~{select_opcode_0}: now also U5.13, U5.2, U5.5
- net ~{select_opcode_1}: now also U14.13, U14.2, U14.5
- net ~{select_opcode_2}: now also U18.13, U18.2, U18.5
- net ~{select_opcode_3}: now also U21.13, U21.2, U21.5
- net ~{select_opcode_4}: now also U22.13, U22.2, U22.5
- net ~{select_opcode_5}: now also U23.13, U23.2, U23.5
- net ~{select_opcode_6}: now also U33.13, U33.2, U33.5
- net ~{select_opcode_7}: now also U34.13, U34.2, U34.5
- net ~{select_opcode_int}: now also U35.13, U35.2, U35.5
- net at U28.3 (C): now also U19.2; no longer U19.4
- net at U12.11 (Cp): now also U19.6; no longer U19.10
- new net: J7.2 (Pin_2), U14.3
- new net: J32.1 (Pin_1), U35.11
- new net: J9.1 (Pin_1), U5.11
- new net: J15.3 (Pin_3), U21.6
- new net: J15.1 (Pin_1), U21.11
- new net: J15.2 (Pin_2), U21.3
- new net: J18.3 (Pin_3), U22.6
- new net: J18.1 (Pin_1), U22.11
- new net: J18.2 (Pin_2), U22.3
- new net: J21.3 (Pin_3), U23.6
- new net: J32.2 (Pin_2), U35.3
- new net: J32.3 (Pin_3), U35.6
- new net: J24.3 (Pin_3), U33.6
- new net: J7.3 (Pin_3), U14.6
- new net: J24.2 (Pin_2), U33.3
- new net: J24.1 (Pin_1), U33.11
- new net: J7.1 (Pin_1), U14.11
- new net: J12.3 (Pin_3), U18.6
- new net: J9.2 (Pin_2), U5.3
- new net: J9.3 (Pin_3), U5.6
- new net: J27.2 (Pin_2), U34.3
- new net: J12.1 (Pin_1), U18.11
- new net: J12.2 (Pin_2), U18.3
- new net: J27.3 (Pin_3), U34.6
- new net: J27.1 (Pin_1), U34.11
- new net: J21.2 (Pin_2), U23.3
- new net: J21.1 (Pin_1), U23.11
- no-connect marks 105 -> 54
Other:
- moved on the sheet: C30, D5, RN3, RN4, RN5, RN7, U19B, U30, U4B
